File: LibreCube PCDU/My version/src/electrical/my_pcdu_v1/my_pcdu_v1.kicad_sch (KiCad schematic)
At the start: 104 parts, among them J1 Conn_01x02, J2 Conn_01x02, J3 Conn_01x02, J4 Conn_01x02, J5 Conn_01x02, J6 Conn_01x02, J7 Conn_01x02, M1 MountingHole, M2 MountingHole, M3 MountingHole, M4 MountingHole, U1 TPS2034, U10 TPS2034, U11 TPS61032, U12 TPS61032, U2 TPS2034, U3 TPS2034, U4 TPS2034, U5 TPS61032, U6 TPS61032, U7 bq24002, U8 bq24002, U9 TPS2034

Commit message: More updates
Parts:
- added D25: LED, Diode_SMD:D_0805_2012Metric, symbol Device:D
- added R19: 1.5k, Resistor_SMD:R_0805_2012Metric, symbol Device:R
- renumbered D26 to D13, D27 to D14, D28 to D15, D29 to D16, D22 to D21, D23 to D22, D24 to D23, D25 to D24, R21 to R11, R22 to R12, R23 to R13, R24 to R14
Connections:
- net +5V: now also H2.25, H2.26, D25.2 (A)
- net +BATT: now also H2.45, H2.46
- net CHARGE: now also H1.31, H1.32
- net GND: now also H1.33, H1.34, H2.29, H2.30, H2.31, H2.32, H2.41, H2.42, H2.43, H2.44, R19.2
- net S2: now also H2.37, H2.38, H2.39, H2.40
- new net: D25.1 (K), R19.1
- no-connect marks 14 -> 90
Other:
- note added: "KillSwitch common"
- note added: "KillSwitch normal open"
- note added: "RBF common"
- note added: "RBF normal open"
- title: (none) -> LibreCube PCDU (LC2201) Schematic
- moved on the sheet: D13, D14, D15, D16, H1, H2, R11, R12, R13, R14

Commit message: Updates
Parts:
- removed BT1, BT2: Battery_Cell, Battery:BatteryHolder_Keystone_1042_1x18650, symbol Device:Battery_Cell
- removed C1, C2, C21, C22, C23, C24, C3, C4, C5, C6, C7, C8: 0.1uF, Capacitor_SMD:C_0805_2012Metric, symbol Device:C
- removed C10, C15, C16, C19, C20, C25, C26, C9: 10uF, Capacitor_SMD:C_0805_2012Metric, symbol Device:C
- removed C11, C12, C27, C28: 2.2uF, Capacitor_SMD:C_0805_2012Metric, symbol Device:C
- removed C13, C14, C29, C30: 220uF, Capacitor_Tantalum_SMD:CP_EIA-7343-31_Kemet-D, symbol Device:C
- removed C17, C18: 0.22uF, Capacitor_SMD:C_0805_2012Metric, symbol Device:C
- removed D1, D10, D11, D12, D2, D21, D22, D23, D24, D3, D4, D5, D6, D7, D8, D9: D_Schottky, Diode_SMD:D_SOD-123, symbol Device:D_Schottky
- removed D13, D14, D15, D16, D17, D18, D19, D20, D25: LED, Diode_SMD:D_0805_2012Metric, symbol Device:D
- removed H1, H2: ESQ-126-39-G-D, ESQ-126-39-G-D:SAMTEC_ESQ-126-39-G-D, symbol ESQ-126-39-G-D:ESQ-126-39-G-D
- removed J1, J2, J3, J4, J5, J6: Conn_01x02, Connector_PinHeader_2.54mm:PinHeader_1x02_P2.54mm_Horizontal, symbol Connector_Generic:Conn_01x02
- removed J7: Conn_01x02, Connector_PinHeader_2.54mm:PinHeader_1x02_P2.54mm_Vertical, symbol Connector_Generic:Conn_01x02
- removed L1, L2, L3, L4: 6.8uH, Inductor_SMD:L_10.4x10.4_H4.8, symbol Device:L
- removed R1, R2, R20, R3, R4: 1M, Resistor_SMD:R_0805_2012Metric, symbol Device:R
- removed R10, R8: 110k, Resistor_SMD:R_0805_2012Metric, symbol Device:R
- removed R11, R12, R13, R14, R15, R16, R17, R18, R19: 1.5k, Resistor_SMD:R_0805_2012Metric, symbol Device:R
- removed R5, R6: 0.1, Resistor_SMD:R_1206_3216Metric, symbol Device:R
- removed R7, R9: 309k, Resistor_SMD:R_0805_2012Metric, symbol Device:R
- removed U1, U10, U2, U3, U4, U9: TPS2034, Package_SO:SO-8_3.9x4.9mm_P1.27mm, symbol mylib:TPS2034
- removed U11, U12, U5, U6: TPS61032, Package_SO:HTSSOP-16-1EP_4.4x5mm_P0.65mm_EP3x3mm, symbol mylib:TPS61032
- removed U7, U8: bq24002, Package_SO:HTSSOP-20-1EP_4.4x6.5mm_P0.65mm_EP2.85x4mm, symbol mylib:bq24002
- added H1, H2: ESQ-126-39-x-D, Connector_PinHeader_2.54mm:PinHeader_2x26_P2.54mm_Vertical, symbol Connector_Generic:Conn_02x26_Odd_Even
Connections:
- net CHARGE: now also H1.31 (Pin_31), H1.32 (Pin_32)
- net ENA_LCL_1: now also H1.45 (Pin_45)
- net ENA_LCL_2: now also H1.47 (Pin_47)
- net ENA_LCL_3: now also H1.49 (Pin_49)
- net ENA_LCL_4: now also H1.51 (Pin_51)
- net GND: now also H1.33 (Pin_33), H1.34 (Pin_34), H2.29 (Pin_29), H2.30 (Pin_30), H2.31 (Pin_31), H2.32 (Pin_32)
- new net 5V: H1.25 (Pin_25), H1.26 (Pin_26), H2.25 (Pin_25), H2.26 (Pin_26)
- new net CAN_A_H: H1.3 (Pin_3)
- new net CAN_A_L: H1.1 (Pin_1)
- new net CAN_B_H: H1.4 (Pin_4)
- new net CAN_B_L: H1.2 (Pin_2)
- new net ENA_LCL_5: H2.33 (Pin_33)
- new net ENA_LCL_6: H2.35 (Pin_35)
- new net ENA_LCL_7: H2.37 (Pin_37)
- new net ENA_LCL_8: H2.39 (Pin_39)
- new net LCL_1: H1.46 (Pin_46)
- new net LCL_2: H1.48 (Pin_48)
- new net LCL_3: H1.50 (Pin_50)
- new net LCL_4: H1.52 (Pin_52)
- new net LCL_5: H2.34 (Pin_34)
- new net LCL_6: H2.36 (Pin_36)
- new net LCL_7: H2.38 (Pin_38)
- new net LCL_8: H2.40 (Pin_40)
- new net UART_A_RX: H1.7 (Pin_7)
- new net UART_A_TX: H1.5 (Pin_5)
- new net UART_B_RX: H1.8 (Pin_8)
- new net UART_B_TX: H1.6 (Pin_6)
- new net UART_C_RX: H1.15 (Pin_15)
- new net UART_C_TX: H1.13 (Pin_13)
- new net UART_D_RX: H1.24 (Pin_24)
- new net UART_D_TX: H1.22 (Pin_22)
- new net VBAT: H2.45 (Pin_45), H2.46 (Pin_46)
- no-connect marks 90 -> 62
Other:
- note removed: "90% charged"
- note removed: "Battery Charger"
- note removed: "Charging"
- note removed: "CubeSat Connector"
- note removed: "KillSwitch common"
- note removed: "KillSwitch normal open"
- note removed: "Power Conditioning Unit"
- note removed: "Power Distribution Unit"
- note removed: "RBF common"
- note removed: "RBF normal open"
- note removed: "Secure Lock"
- note removed: "Solar Array Input"
- note removed: "Solar Array Regulator"
- note removed: "System Power Regulator"
- note removed: "System Power Switch"
- title: LibreCube PCDU (LC2201) Schematic -> (none)
