File: LibreCube PCDU/My version/src/electrical/my_pcdu_v1.kicad_sch (KiCad schematic)
At the start: 6 parts, among them M1 MountingHole, M2 MountingHole, M3 MountingHole, M4 MountingHole

Commit message: Updates
Parts:
- added BT1, BT2: Battery_Cell, Battery:BatteryHolder_Keystone_1042_1x18650, symbol Device:Battery_Cell
- added C1, C11, C12, C17, C18, C2, C7, C8: 10uF, Capacitor_SMD:C_0805_2012Metric, symbol Device:C
- added C10, C9: 0.22uF, Capacitor_SMD:C_0805_2012Metric, symbol Device:C
- added C13, C14, C15, C16, C23, C24, C25, C26, C27, C28, C29, C30: 0.1uF, Capacitor_SMD:C_0805_2012Metric, symbol Device:C
- added C19, C20, C3, C4: 2.2uF, Capacitor_SMD:C_0805_2012Metric, symbol Device:C
- added C21, C22, C5, C6: 220uF, Capacitor_Tantalum_SMD:CP_EIA-7343-31_Kemet-D, symbol Device:C
- added D1, D10, D11, D12, D17, D18, D19, D2, D20, D3, D4, D5, D6, D7, D8, D9: D_Schottky, Diode_SMD:D_SOD-123, symbol Device:D_Schottky
- added D13, D14, D15, D16, D21, D22, D23, D24, D25: LED, Diode_SMD:D_0805_2012Metric, symbol Device:D
- added J1, J2, J3, J4, J5, J6: Conn_01x02, Connector_PinHeader_2.54mm:PinHeader_1x02_P2.54mm_Horizontal, symbol Connector_Generic:Conn_01x02
- added J7: Conn_01x02, Connector_PinHeader_2.54mm:PinHeader_1x02_P2.54mm_Vertical, symbol Connector_Generic:Conn_01x02
- added L1, L2, L3, L4: 6.8uH, Inductor_SMD:L_10.4x10.4_H4.8, symbol Device:L
- added R1, R2: 0.1, Resistor_SMD:R_1206_3216Metric, symbol Device:R
- added R10, R16, R17, R18, R19, R20, R7, R8, R9: 1.5k, Resistor_SMD:R_0805_2012Metric, symbol Device:R
- added R11, R12, R13, R14, R15: 1M, Resistor_SMD:R_0805_2012Metric, symbol Device:R
- added R3, R5: 309k, Resistor_SMD:R_0805_2012Metric, symbol Device:R
- added R4, R6: 110k, Resistor_SMD:R_0805_2012Metric, symbol Device:R
- added U1, U2, U7, U8: TPS61032, Package_SO:HTSSOP-16-1EP_4.4x5mm_P0.65mm_EP3x3mm, symbol mylib:TPS61032
- added U10, U11, U12, U5, U6, U9: TPS2034, Package_SO:SO-8_3.9x4.9mm_P1.27mm, symbol mylib:TPS2034
- added U3, U4: bq24002, Package_SO:HTSSOP-20-1EP_4.4x6.5mm_P0.65mm_EP2.85x4mm, symbol mylib:bq24002
Connections:
- net ENA_LCL_8 is gone; now on net S2: H2.39 (Pin_39)
- net LCL_7 is gone; now on net S2: H2.38 (Pin_38)
- net LCL_8 is gone; now on net S2: H2.40 (Pin_40)
- net 5V: no longer H2.25 (Pin_25), H2.26 (Pin_26)
- net CHARGE: now also C1.1, C2.1, D1.1 (K), D10.1 (K), D11.1 (K), D12.1 (K), D2.1 (K), D3.1 (K), D4.1 (K), D5.1 (K), D6.1 (K), D7.1 (K), D8.1 (K), D9.1 (K), L1.2, L2.2, U1.6 (VBAT), U1.9 (EN), U2.6 (VBAT), U2.9 (EN)
- net ENA_LCL_1: now also H1.51 (Pin_51), R12.1, U9.4 (EN); no longer H1.45 (Pin_45)
- net ENA_LCL_2: now also H1.49 (Pin_49), R13.1, U10.4 (EN); no longer H1.47 (Pin_47)
- net ENA_LCL_3: now also H1.47 (Pin_47), R14.1, U11.4 (EN); no longer H1.49 (Pin_49)
- net ENA_LCL_4: now also H1.45 (Pin_45), R15.1, U12.4 (EN); no longer H1.51 (Pin_51)
- net GND: now also H2.41 (Pin_41), H2.42 (Pin_42), H2.43 (Pin_43), H2.44 (Pin_44), BT1.2 (-), BT2.2 (-), C1.2, C10.2, C11.2, C12.2, C13.2, C14.2, C15.2, C16.2, C17.2, C18.2, C19.2, C2.2, C20.2, C21.2, C22.2, C23.2, C24.2, C25.2, C26.2, C27.2, C28.2, C29.2, C3.2, C30.2, C4.2, C5.2, C6.2, C7.2, C8.2, C9.2, J1.2 (Pin_2), J2.2 (Pin_2), J3.2 (Pin_2), J4.2 (Pin_2), J5.2 (Pin_2), J6.2 (Pin_2), J7.2 (Pin_2), R12.2, R13.2, R14.2, R15.2, R16.2, R17.2, R18.2, R19.2, R20.2, R4.2, R6.2, U1.11 (GND), U1.17 (PAD), U1.3 (PGND), U1.4 (PGND), U1.5 (PGND), U1.7 (LBI), U1.8 (SYNC), U10.1 (GND), U11.1 (GND), U12.1 (GND), U2.11 (GND), U2.17 (PAD), U2.3 (PGND), U2.4 (PGND), U2.5 (PGND), U2.7 (LBI), U2.8 (SYNC), U3.10 (GND), U3.13 (TMR_SEL), U3.16 (AGND), U4.10 (GND), U4.13 (TMR_SEL), U4.16 (AGND), U5.1 (GND), U6.1 (GND), U7.11 (GND), U7.17 (PAD), U7.3 (PGND), U7.4 (PGND), U7.5 (PGND), U7.7 (LBI), U7.8 (SYNC), U8.11 (GND), U8.17 (PAD), U8.3 (PGND), U8.4 (PGND), U8.5 (PGND), U8.7 (LBI), U8.8 (SYNC), U9.1 (GND)
- net ENA_LCL_5: no longer names the net of H2.33 (Pin_33)
- net ENA_LCL_6: no longer names the net of H2.35 (Pin_35)
- net ENA_LCL_7 renamed S2
- net S2: now also J7.1 (Pin_1), R11.2, U5.4 (EN), U6.4 (EN)
- net LCL_1 renamed PWR_LCL_4
- net PWR_LCL_4: now also C30.1, D24.2 (A), U12.6 (OUT), U12.7 (OUT), U12.8 (OUT)
- net LCL_2 renamed PWR_LCL_3
- net PWR_LCL_3: now also C29.1, D23.2 (A), U11.6 (OUT), U11.7 (OUT), U11.8 (OUT)
- net LCL_3 renamed PWR_LCL_2
- net PWR_LCL_2: now also C28.1, D22.2 (A), U10.6 (OUT), U10.7 (OUT), U10.8 (OUT)
- net LCL_4 renamed PWR_LCL_1
- net PWR_LCL_1: now also C27.1, D21.2 (A), U9.6 (OUT), U9.7 (OUT), U9.8 (OUT)
- net LCL_5: no longer names the net of H2.34 (Pin_34)
- net LCL_6: no longer names the net of H2.36 (Pin_36)
- net VBAT renamed +BATT
- net +BATT: now also BT1.1 (+), BT2.1 (+), C11.1, C12.1, D19.2 (A), D20.2 (A), U3.17 (VSENSE), U3.18 (OUT`), U3.19 (OUT), U4.17 (VSENSE), U4.18 (OUT`), U4.19 (OUT)
- new net: D1.2 (A), D2.2 (A), J1.1 (Pin_1)
- new net: C3.1, C4.1, C5.1, C6.1, C7.1, C8.1, D17.2 (A), D18.2 (A), R1.2, R10.1, R2.2, R3.1, R5.1, R7.1, R8.1, R9.1, U1.13 (VOUT), U1.14 (VOUT), U1.15 (VOUT), U2.13 (VOUT), U2.14 (VOUT), U2.15 (VOUT), U3.4 (VCC), U3.8 (EN), U3.9 (VSEL), U4.4 (VCC), U4.8 (EN), U4.9 (VSEL)
- new net: L2.1, U2.1 (SW), U2.2 (SW)
- new net: R3.2, R4.1, U3.7 (APG/THERM)
- new net: D21.1 (K), R16.1
- new net: C9.1, U3.12 (CR)
- new net: D25.1 (K), R20.1
- new net: D14.1 (K), U4.15 (STAT2)
- new net: D14.2 (A), R8.2
- new net: D24.1 (K), R19.1
- new net: R5.2, R6.1, U4.7 (APG/THERM)
- new net: L1.1, U1.1 (SW), U1.2 (SW)
- new net: D11.2 (A), D12.2 (A), J6.1 (Pin_1)
- new net: D5.2 (A), D6.2 (A), J3.1 (Pin_1)
- new net: D15.2 (A), R9.2
- new net: C10.1, U4.12 (CR)
- new net: D16.1 (K), U4.14 (STAT1)
- new net: R2.1, U4.2 (IN), U4.3 (IN), U4.5 (ISNS)
- new net: L4.1, U8.1 (SW), U8.2 (SW)
- new net: C15.1, C16.1, C17.1, C18.1, L3.2, L4.2, U5.6 (OUT), U5.7 (OUT), U5.8 (OUT), U6.6 (OUT), U6.7 (OUT), U6.8 (OUT), U7.6 (VBAT), U7.9 (EN), U8.6 (VBAT), U8.9 (EN)
- new net: D16.2 (A), R10.2
- new net: D10.2 (A), D9.2 (A), J5.1 (Pin_1)
- new net: D7.2 (A), D8.2 (A), J4.1 (Pin_1)
- new net: D13.1 (K), U3.15 (STAT2)
- new net: D13.2 (A), R7.2
- new net: D23.1 (K), R18.1
- new net: L3.1, U7.1 (SW), U7.2 (SW)
- new net: D22.1 (K), R17.1
- new net: D3.2 (A), D4.2 (A), J2.1 (Pin_1)
- new net: D15.1 (K), U3.14 (STAT1)
- new net: R1.1, U3.2 (IN), U3.3 (IN), U3.5 (ISNS)
- new net +5V: C19.1, C20.1, C21.1, C22.1, C23.1, C24.1, C25.1, C26.1, D25.2 (A), H2.25 (Pin_25), H2.26 (Pin_26), U10.2 (IN), U10.3 (IN), U11.2 (IN), U11.3 (IN), U12.2 (IN), U12.3 (IN), U7.13 (VOUT), U7.14 (VOUT), U7.15 (VOUT), U8.13 (VOUT), U8.14 (VOUT), U8.15 (VOUT), U9.2 (IN), U9.3 (IN)
- new net Semi_Regulated_Bus: C13.1, C14.1, D17.1 (K), D18.1 (K), D19.1 (K), D20.1 (K), R11.1, U5.2 (IN), U5.3 (IN), U6.2 (IN), U6.3 (IN)
- no-connect marks 62 -> 75
Other:
- note added: "90% charged"
- note added: "Battery Charger"
- note added: "Charging"
- note added: "CubeSat Connector"
- note added: "KillSwitch common"
- note added: "KillSwitch normal open"
- note added: "Power Conditioning Unit"
- note added: "Power Distribution Unit"
- note added: "RBF common"
- note added: "RBF normal open"
- note added: "Secure Lock"
- note added: "Solar Array Input"
- note added: "Solar Array Regulator"
- note added: "System Power Regulator"
- note added: "System Power Switch"
- company: (none) -> Power Electronics and PCB Engineer
- title: (none) -> LibreCube PCDU 4-Layer (LC2201)
- moved on the sheet: H1, H2, M1, M2, M3, M4

Commit message: Updates
Parts:
- removed U4: bq24002, Package_SO:HTSSOP-20-1EP_4.4x6.5mm_P0.65mm_EP2.85x4mm, symbol mylib:bq24002
- added U8: bq24002, Package_SO:HTSSOP-20-1EP_4.4x6.5mm_P0.65mm_EP2.85x4mm, symbol mylib:bq24002
- renumbered C23 to C1, C2 to C10, C3 to C11, C4 to C12, C5 to C13, C6 to C14, C7 to C15, C8 to C16, C9 to C17, C10 to C18, C11 to C19, C24 to C2, C12 to C20, C13 to C21, C14 to C22, C15 to C23, C16 to C24, C17 to C25, C18 to C26, C19 to C27, C20 to C28, C21 to C29, C25 to C3, C22 to C30, C26 to C4, C27 to C5, C28 to C6, C29 to C7, C30 to C8, C1 to C9, D21 to D13, D22 to D14, D23 to D15, D24 to D16, D13 to D17, D14 to D18, D15 to D19, D16 to D20, D25 to D21, D17 to D22, D18 to D23, D19 to D24, D20 to D25, R12 to R1, R4 to R10, R5 to R11, R6 to R12, R18 to R13, R19 to R14, R7 to R15, R8 to R16, R9 to R17, R10 to R18, R20 to R19, R13 to R2, R11 to R20, R14 to R3, R15 to R4, R16 to R5, R1 to R6, R2 to R7, R17 to R8, R3 to R9, U9 to U1, U6 to U10, U7 to U11, U8 to U12, U10 to U2, U11 to U3, U12 to U4, U1 to U5, U2 to U6, U3 to U7, U5 to U9
Connections:
- net 5V is gone; now on net +5V: H1.25 (Pin_25), H1.26 (Pin_26)
- net +BATT: now also U8.17 (VSENSE), U8.18 (OUT`), U8.19 (OUT)
- net GND: now also U8.10 (GND), U8.13 (TMR_SEL), U8.16 (AGND)
- net at C11.1, C12.1, C13.1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: now also U8.4 (VCC), U8.8 (EN), U8.9 (VSEL)
- net at D18.1 (K): now also U8.15 (STAT2)
- net at R11.2, R12.1: now also U8.7 (APG/THERM)
- net at C18.1: now also U8.12 (CR)
- net at D20.1 (K): now also U8.14 (STAT1)
- net at R7.1: now also U8.2 (IN), U8.3 (IN), U8.5 (ISNS)
- net CAN_A_H: no longer names the net of H1.3 (Pin_3)
- net CAN_A_L: no longer names the net of H1.1 (Pin_1)
- net CAN_B_H: no longer names the net of H1.4 (Pin_4)
- net CAN_B_L: no longer names the net of H1.2 (Pin_2)
- net UART_A_RX: no longer names the net of H1.7 (Pin_7)
- net UART_A_TX: no longer names the net of H1.5 (Pin_5)
- net UART_B_RX: no longer names the net of H1.8 (Pin_8)
- net UART_B_TX: no longer names the net of H1.6 (Pin_6)
- net UART_C_RX: no longer names the net of H1.15 (Pin_15)
- net UART_C_TX: no longer names the net of H1.13 (Pin_13)
- net UART_D_RX: no longer names the net of H1.24 (Pin_24)
- net UART_D_TX: no longer names the net of H1.22 (Pin_22)
- no-connect marks 75 -> 87
Other:
- moved on the sheet: D17, D18, D19, D20, R15, R16

Commit message: Uploaded PCDUv2
Connections:
- net ENA_LCL_1: now also H1.45 (Pin_45); no longer H1.51 (Pin_51)
- net ENA_LCL_2: now also H1.47 (Pin_47); no longer H1.49 (Pin_49)
- net ENA_LCL_3: now also H1.49 (Pin_49); no longer H1.47 (Pin_47)
- net ENA_LCL_4: now also H1.51 (Pin_51); no longer H1.45 (Pin_45)
- net PWR_LCL_1: now also D16.2 (A), H1.46 (Pin_46); no longer D13.2 (A), H1.52 (Pin_52)
- net PWR_LCL_2: now also D15.2 (A), H1.48 (Pin_48); no longer D14.2 (A), H1.50 (Pin_50)
- net PWR_LCL_3: now also D14.2 (A), H1.50 (Pin_50); no longer D15.2 (A), H1.48 (Pin_48)
- net PWR_LCL_4: now also D13.2 (A), H1.52 (Pin_52); no longer D16.2 (A), H1.46 (Pin_46)

Commit message: More updates
Parts:
- removed D13, D14, D15, D16: LED, Diode_SMD:D_0805_2012Metric, symbol Device:D
- removed R13, R14: 1.5k, Resistor_SMD:R_0805_2012Metric, symbol Device:R
- added C31, C32, C33, C34, C35, C36, C37, C38: 0.1uF, Capacitor_SMD:C_0805_2012Metric, symbol Device:C
- added J8: USB_C_Receptacle_PowerOnly_6P, Connector_USB:USB_C_Receptacle_GCT_USB4125-xx-x-0190_6P_TopMnt_Horizontal, symbol Connector:USB_C_Receptacle_PowerOnly_6P
- added R21, R22, R23, R24: 1M, Resistor_SMD:R_0805_2012Metric, symbol Device:R
- added U13, U14, U15, U16: TPS2034, Package_SO:SO-8_3.9x4.9mm_P1.27mm, symbol mylib:TPS2034
- R5, R8: value 1.5k -> 5.1k
Connections:
- net +5V: now also C31.1, C32.1, C33.1, C34.1, U13.2 (IN), U13.3 (IN), U14.2 (IN), U14.3 (IN), U15.2 (IN), U15.3 (IN), U16.2 (IN), U16.3 (IN)
- net CHARGE: now also J8.A9 (VBUS), J8.B9 (VBUS)
- net GND: now also H2.50 (Pin_50), H2.52 (Pin_52), C31.2, C32.2, C33.2, C34.2, C35.2, C36.2, C37.2, C38.2, J8.A12 (GND), J8.B12 (GND), J8.S1 (SHIELD), R21.2, R22.2, R23.2, R24.2, U13.1 (GND), U14.1 (GND), U15.1 (GND), U16.1 (GND); no longer H2.41 (Pin_41), H2.42 (Pin_42), H2.43 (Pin_43), H2.44 (Pin_44)
- net ENA_LCL_5: now reaches H2.33 (Pin_33)
- net ENA_LCL_5: now also R21.1, U13.4 (EN)
- net PWR_LCL_5: now reaches H2.34 (Pin_34)
- net PWR_LCL_5: now also C35.1, U13.6 (OUT), U13.7 (OUT), U13.8 (OUT)
- net ENA_LCL_6: now reaches H2.35 (Pin_35)
- net ENA_LCL_6: now also R22.1, U14.4 (EN)
- net PWR_LCL_6: now reaches H2.36 (Pin_36)
- net PWR_LCL_6: now also C36.1, U14.6 (OUT), U14.7 (OUT), U14.8 (OUT)
- net KS_OPEN: now reaches H2.49 (Pin_49)
- net KS_OPEN: now also H2.51 (Pin_51), J7.1 (Pin_1), R20.2, U10.4 (EN), U9.4 (EN)
- net at R5.1: now also J8.B5 (CC2)
- net at R8.1: now also J8.A5 (CC1)
- removed net S2: H2.37 (Pin_37), H2.38 (Pin_38), H2.39 (Pin_39), H2.40 (Pin_40), J7.1 (Pin_1), R20.2, U10.4 (EN), U9.4 (EN)
- new net ENA_LCL_7: H2.37 (Pin_37), R23.1, U15.4 (EN)
- new net ENA_LCL_8: H2.39 (Pin_39), R24.1, U16.4 (EN)
- new net PWR_LCL_7: C37.1, H2.38 (Pin_38), U15.6 (OUT), U15.7 (OUT), U15.8 (OUT)
- new net PWR_LCL_8: C38.1, H2.40 (Pin_40), U16.6 (OUT), U16.7 (OUT), U16.8 (OUT)
Other:
- note added: "KS Ground"
- note added: "KS Open"
- note added: "RBF Ground"
- note added: "RBF Open"
- note removed: "KillSwitch common"
- note removed: "KillSwitch normal open"
- note removed: "RBF common"
- note removed: "RBF normal open"
- moved on the sheet: C1, C2, C3, C4, C5, C6, C7, C8, H2, R1, R2, R3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

Commit message: New components
Parts:
- added U17, U18: TPS61023DRLR, TPS61023DRLR:DRL0006A, symbol TPS61023DRLR:TPS61023DRLR
- added U19, U20: TPS61232DRCR, TPS61232DRCR:VREG_TPS61232DRCR, symbol TPS61232DRCR:TPS61232DRCR
Connections:
- new net: U20.1 (SW), U20.2 (SW)
- new net: U20.11 (GND), U20.11_1 (GND), U20.11_2 (GND), U20.11_3 (GND), U20.11_4 (GND)
- new net: U20.3 (VOUT), U20.4 (VOUT)
- new net: U19.1 (SW), U19.2 (SW)
- new net: U19.11 (GND), U19.11_1 (GND), U19.11_2 (GND), U19.11_3 (GND), U19.11_4 (GND)
- new net: U19.3 (VOUT), U19.4 (VOUT)
Other:
- moved on the sheet: J8, M1, M2, M3, M4, R5, R8

Commit message: PCDU updates
Parts:
- removed C29, C30: 220uF, Capacitor_Tantalum_SMD:CP_EIA-7343-31_Kemet-D, symbol Device:C
- removed D17, D18, D19, D20: LED, Diode_SMD:D_0805_2012Metric, symbol Device:D
- removed L3, L4: 6.8uH, Inductor_SMD:L_10.4x10.4_H4.8, symbol Device:L
- removed U11, U12, U5, U6: TPS61032, Package_SO:HTSSOP-16-1EP_4.4x5mm_P0.65mm_EP3x3mm, symbol mylib:TPS61032
- removed U18: TPS61023DRLR, TPS61023DRLR:DRL0006A, symbol TPS61023DRLR:TPS61023DRLR
- removed U7, U8: bq24002, Package_SO:HTSSOP-20-1EP_4.4x6.5mm_P0.65mm_EP2.85x4mm, symbol mylib:bq24002
- added D13, D15: Red, LED_SMD:LED_0805_2012Metric_Pad1.15x1.40mm_HandSolder, symbol Device:LED
- added D14, D16: Green, LED_SMD:LED_0805_2012Metric_Pad1.15x1.40mm_HandSolder, symbol Device:LED
- added R13, R25, R26, R29: 100k, Resistor_SMD:R_0805_2012Metric_Pad1.20x1.40mm_HandSolder, symbol Device:R
- added R14, R27, R28: 1k5, Resistor_SMD:R_0805_2012Metric_Pad1.20x1.40mm_HandSolder, symbol Device:R
- added R30: 10k, Resistor_SMD:R_0805_2012Metric_Pad1.20x1.40mm_HandSolder, symbol Device:R
- added R31: 820Ω, Resistor_SMD:R_0805_2012Metric_Pad1.20x1.40mm_HandSolder, symbol Device:R
- added R32: 37k4, Resistor_SMD:R_0805_2012Metric_Pad1.20x1.40mm_HandSolder, symbol Device:R
- added U5, U7: BQ24032ARHLRG4, BQ24032ARHLRG4:IC_MSP430FR2522IRHLR, symbol BQ24032ARHLRG4:BQ24032ARHLRG4
- added U6: TPS61023DRLR, TPS61023DRLR:DRL0006A, symbol TPS61023DRLR:TPS61023DRLR
- C10, C19, C20, C9: footprint Capacitor_SMD:C_0805_2012Metric -> Capacitor_SMD:C_0805_2012Metric_Pad1.18x1.45mm_HandSolder
- C11, C12, C27, C28: value 2.2uF -> 10uF; footprint Capacitor_SMD:C_0805_2012Metric -> Capacitor_SMD:C_0805_2012Metric_Pad1.18x1.45mm_HandSolder
- C13, C14: value 220uF -> 22uF; footprint Capacitor_Tantalum_SMD:CP_EIA-7343-31_Kemet-D -> Capacitor_SMD:C_0805_2012Metric_Pad1.18x1.45mm_HandSolder
- C15, C16: value 10uF -> 22uF; footprint Capacitor_SMD:C_0805_2012Metric -> Capacitor_SMD:C_0805_2012Metric_Pad1.18x1.45mm_HandSolder
- C17, C18: value 0.22uF -> 10u; footprint Capacitor_SMD:C_0805_2012Metric -> Capacitor_SMD:C_1206_3216Metric_Pad1.33x1.80mm_HandSolder
- C25, C26: value 10uF -> 10u; footprint Capacitor_SMD:C_0805_2012Metric -> Capacitor_SMD:C_1206_3216Metric_Pad1.33x1.80mm_HandSolder
- L1, L2: value 6.8uH -> 1uH; footprint Inductor_SMD:L_10.4x10.4_H4.8 -> Inductor_SMD:L_Coilcraft_XxL4040
- R10: value 110k -> 750k; footprint Resistor_SMD:R_0805_2012Metric -> Resistor_SMD:R_0805_2012Metric_Pad1.20x1.40mm_HandSolder
- R11: value 309k -> 10k; footprint Resistor_SMD:R_0805_2012Metric -> Resistor_SMD:R_0805_2012Metric_Pad1.20x1.40mm_HandSolder
- R12: value 110k -> 100k; footprint Resistor_SMD:R_0805_2012Metric -> Resistor_SMD:R_0805_2012Metric_Pad1.20x1.40mm_HandSolder
- R15: value 1.5k -> 1k5; footprint Resistor_SMD:R_0805_2012Metric -> Resistor_SMD:R_0805_2012Metric_Pad1.20x1.40mm_HandSolder
- R16: value 1.5k -> 820Ω; footprint Resistor_SMD:R_0805_2012Metric -> Resistor_SMD:R_0805_2012Metric_Pad1.20x1.40mm_HandSolder
- R17: value 1.5k -> 37k4; footprint Resistor_SMD:R_0805_2012Metric -> Resistor_SMD:R_0805_2012Metric_Pad1.20x1.40mm_HandSolder
- R18: value 1.5k -> 100k; footprint Resistor_SMD:R_0805_2012Metric -> Resistor_SMD:R_0805_2012Metric_Pad1.20x1.40mm_HandSolder
- R6: value 0.1 -> 750k; footprint Resistor_SMD:R_1206_3216Metric -> Resistor_SMD:R_0805_2012Metric_Pad1.20x1.40mm_HandSolder
- R7: value 0.1 -> 100k; footprint Resistor_SMD:R_1206_3216Metric -> Resistor_SMD:R_0805_2012Metric_Pad1.20x1.40mm_HandSolder
- R9: value 309k -> 100k; footprint Resistor_SMD:R_0805_2012Metric -> Resistor_SMD:R_0805_2012Metric_Pad1.20x1.40mm_HandSolder
Connections:
- net +5V: no longer C27.1, C28.1
- net +BATT: now also C27.1, U5.5 (BAT-1), U5.6 (BAT), U7.5 (BAT-1), U7.6 (BAT); no longer C19.1, D24.2 (A), D25.2 (A)
- net CHARGE: now also C11.1, C12.1, L1.1, L2.1, U17.2 (EN), U17.3 (VIN), U6.2 (EN), U6.3 (VIN); no longer L1.2, L2.2
- net GND: now also R11.2, R16.2, R17.2, R7.2, R9.2, U17.4 (GND), R30.2, R31.2, R32.2, U5.11 (VSS), U6.4 (GND), U7.11 (VSS); no longer R10.2, R12.2
- net at C13.1, C14.1, C15.1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: now also C17.1, C18.1, C25.1, C26.1, R10.2, R12.1, U17.6 (VOUT), R13.1, R14.1, R25.1, R26.1, R27.1, R28.1, R29.1, U5.4 (AC), U6.6 (VOUT), U7.4 (AC); no longer C11.1, C12.1, R11.1, R16.1, R17.1, R7.2, R9.1
- net at R10.1: now also R9.1, U6.1 (FB); no longer R9.2
- net at U17.1 (FB): now also R6.1, R7.1
- net at U17.5 (SW): now also L1.2
- net at C23.1, C24.1, U10.6 (OUT)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: no longer C25.1, C26.1
- net at R18.2: now also U7.7 (ISET2)
- net at R15.2: now also D14.2 (A)
- new net: R16.1, U7.10 (ISET1)
- new net: D15.2 (A), R27.2
- new net: R26.2, U5.9 (CE)
- new net: C19.1, C28.1, D24.2 (A), D25.2 (A), U5.15 (OUT-1), U5.16 (OUT), U5.17 (OUT-2), U7.15 (OUT-1), U7.16 (OUT), U7.17 (OUT-2)
- new net: L2.2, U6.5 (SW)
- new net: U7.1 (LDO), U7.14 (TMR)
- new net: R11.1, U7.12 (TS)
- new net: R17.1, U7.13 (DPPM)
- new net: U7.18 (~{ACPG}), U7.19 (~{USBPG})
- new net: D13.1 (K), U7.2 (STAT1)
- new net: D14.1 (K), U7.3 (STAT2)
- new net: R12.2, U7.8 (PSEL)
- new net: R13.2, U7.9 (CE)
- new net: D13.2 (A), R14.2
- new net: R32.1, U5.13 (DPPM)
- new net: D16.2 (A), R28.2
- new net: R31.1, U5.10 (ISET1)
- new net: D16.1 (K), U5.3 (STAT2)
- new net: R29.2, U5.7 (ISET2)
- new net: D15.1 (K), U5.2 (STAT1)
- new net: R25.2, U5.8 (PSEL)
- new net: U5.1 (LDO), U5.14 (TMR)
- new net: R30.1, U5.12 (TS)
- new net: U5.18 (~{ACPG}), U5.19 (~{USBPG})
- no-connect marks 87 -> 80
Other:
- note removed: "90% charged"
- note removed: "Charging"
- moved on the sheet: BT1, BT2, D22, D23, D24, D25, U17, U19, U20

Commit message: PCB Layout
Parts:
- removed U20: TPS61232DRCR, TPS61232DRCR:VREG_TPS61232DRCR, symbol TPS61232DRCR:TPS61232DRCR
- removed U5: BQ24032ARHLRG4, BQ24032ARHLRG4:IC_MSP430FR2522IRHLR, symbol BQ24032ARHLRG4:BQ24032ARHLRG4
- added C37, C38, C41, C42, C43, C44, C45, C46: 22uF, Capacitor_SMD:C_0805_2012Metric_Pad1.18x1.45mm_HandSolder, symbol Device:C
- added C39, C40: 10nF, Capacitor_SMD:C_0805_2012Metric_Pad1.18x1.45mm_HandSolder, symbol Device:C
- added L3, L4: 1uH, Inductor_SMD:L_Coilcraft_XAL4040-XXX, symbol Device:L
- added U12: BQ24032ARHLRG4, BQ24032ARHLRG4:IC_MSP430FR2522IRHLR, symbol BQ24032ARHLRG4:BQ24032ARHLRG4
- added U16: TPS61232DRCR, TPS61232DRCR:VREG_TPS61232DRCR, symbol TPS61232DRCR:TPS61232DRCR
- L1, L2: footprint Inductor_SMD:L_Coilcraft_XxL4040 -> Inductor_SMD:L_Coilcraft_XAL4040-XXX
- renumbered C6 to C10, C7 to C11, C8 to C12, C35 to C13, C36 to C14, C37 to C15, C38 to C16, C9 to C17, C11 to C18, C10 to C19, C12 to C20, C13 to C21, C15 to C22, C14 to C23, C16 to C24, C17 to C25, C25 to C26, C18 to C27, C26 to C28, C20 to C29, C27 to C30, C19 to C31, C28 to C32, C21 to C33, C22 to C34, C23 to C35, C24 to C36, C31 to C5, C32 to C6, C33 to C7, C34 to C8, C5 to C9, D22 to D17, D23 to D18, D21 to D19, D24 to D20, D25 to D21, R9 to R10, R6 to R11, R10 to R12, R12 to R13, R13 to R14, R14 to R15, R15 to R16, R18 to R17, R25 to R18, R26 to R19, R27 to R20, R28 to R21, R29 to R22, R11 to R23, R30 to R24, R16 to R25, R31 to R26, R17 to R27, R32 to R28, R19 to R29, R20 to R30, R5 to R31, R8 to R32, R21 to R5, R22 to R6, R23 to R7, R24 to R8, R7 to R9, U6 to U10, U7 to U11, U9 to U13, U10 to U14, U19 to U15, U13 to U5, U14 to U6, U15 to U7, U16 to U8, U17 to U9
Connections:
- net +5V: now also U15.3 (VOUT), U15.4 (VOUT), U15.7 (FB), C41.1, C42.1, C43.1, C44.1, C45.1, C46.1, U16.3 (VOUT), U16.4 (VOUT), U16.7 (FB)
- net +BATT: now also U12.5 (BAT-1), U12.6 (BAT)
- net GND: now also U11.21 (PwrPad), U15.11 (GND), U15.11_1 (GND), U15.11_2 (GND), U15.11_3 (GND), U15.11_4 (GND), C37.2, C38.2, C39.2, C40.2, C41.2, C42.2, C43.2, C44.2, C45.2, C46.2, U12.11 (VSS), U12.21 (PwrPad), U16.11 (GND), U16.11_1 (GND), U16.11_2 (GND), U16.11_3 (GND), U16.11_4 (GND)
- net at C21.1, C22.1, C23.1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: now also U12.4 (AC)
- net at R19.2: now also U12.9 (CE)
- net at C31.1, C32.1, D20.2 (A)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: now also U12.15 (OUT-1), U12.16 (OUT), U12.17 (OUT-2)
- net at C35.1, C36.1, U13.6 (OUT)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: now also U15.10 (VIN), U15.9 (EN), C37.1, C38.1, L3.1, L4.1, U16.10 (VIN), U16.9 (EN)
- net at R28.1: now also U12.13 (DPPM)
- net at U15.1 (SW), U15.2 (SW): now also L3.2
- net at U15.6 (SS): now also C39.1
- net at R26.1: now also U12.10 (ISET1)
- net at D16.1 (K): now also U12.3 (STAT2)
- net at R22.2: now also U12.7 (ISET2)
- net at D15.1 (K): now also U12.2 (STAT1)
- net at R18.2: now also U12.8 (PSEL)
- net at R24.1: now also U12.12 (TS)
- new net: U12.1 (LDO), U12.14 (TMR)
- new net: U12.18 (~{ACPG}), U12.19 (~{USBPG})
- new net: L4.2, U16.1 (SW), U16.2 (SW)
- new net: C40.1, U16.6 (SS)
- no-connect marks 80 -> 84
Other:
- moved on the sheet: U15

Commit message: Updates
Connections:
- net VIN: now reaches C21.1, C22.1, C23.1, C24.1, C25.1, C26.1, C27.1, C28.1, D17.2 (A), D18.2 (A), R11.2, R12.2, R13.1, R14.1, R15.1, R16.1, R17.1, R18.1, R19.1, R20.1, R21.1, R22.1, U10.6 (VOUT), U11.4 (AC), U12.4 (AC), U9.6 (VOUT)
- net VOUT: now reaches C31.1, C32.1, D20.2 (A), D21.2 (A), U11.15 (OUT-1), U11.16 (OUT), U11.17 (OUT-2), U12.15 (OUT-1), U12.16 (OUT), U12.17 (OUT-2)
Changed lines of the file:
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@@
+		)
+	)
+	(label "VIN"
+		(at 349.25 133.35 180)
+		(fields_autoplaced yes)
+		(effects
+			(font
+				(size 1.27 1.27)
+			)
+			(justify right bottom)
+		)
+	)
+	(label "VIN"
+		(at 349.25 196.85 180)
+		(fields_autoplaced yes)
+		(effects
+			(font
+				(size 1.27 1.27)
+			)
+			(justify right bottom)
+		)
+	)
+	(label "VOUT"
+		(at 384.81 133.35 0)
+		(fields_autoplaced yes)
+		(effects
+			(font
+				(size 1.27 1.27)
+			)
+			(justify left bottom)
+		)
+	)
+	(label "VOUT"
+		(at 384.81 196.85 0)
+		(fields_autoplaced yes)
+		(effects
+			(font
+				(size 1.27 1.27)
+			)
+			(justify left bottom)
 		)
 	)
