File: LibreCube PCDU/My version/src/electrical/my_pcdu_v1.kicad_sch (KiCad schematic)
At the start: 135 parts, among them J1 Conn_01x02, J2 Conn_01x02, J3 Conn_01x02, J4 Conn_01x02, J5 Conn_01x02, J6 Conn_01x02, J7 Conn_01x02, J8 USB_C_Receptacle_PowerOnly_6P, M1 MountingHole, M2 MountingHole, M3 MountingHole, M4 MountingHole, U1 TPS2034, U10 TPS61023DRLR, U11 BQ24032ARHLRG4, U12 BQ24032ARHLRG4, U13 TPS2034, U14 TPS2034, U15 TPS61232DRCR, U16 TPS61232DRCR, U2 TPS2034, U3 TPS2034, U4 TPS2034, U5 TPS2034, U6 TPS2034, U7 TPS2034, U8 TPS2034, U9 TPS61023DRLR

Commit message: EPS Routing
Connections:
- net CHARGE: no longer C17.1, C19.1, L1.1, U9.2 (EN), U9.3 (VIN)
- net GND: no longer C17.2, C19.2, C21.2, C23.2, R9.2, U9.4 (GND)
- net VIN: now also U9.3 (VIN); no longer C21.1, C23.1, R11.2, U9.6 (VOUT)
- net at U9.5 (SW): no longer L1.2
- now unconnected: R11.1, R9.1, U9.1 (FB)
- no-connect marks 84 -> 85
Other:
- moved on the sheet: C17, C19, C21, C23, L1, R11, R9, U9

Commit message: updates
Connections:
- net CHARGE: now also C17.1, C19.1, L1.1, U9.2 (EN), U9.3 (VIN)
- net GND: now also C17.2, C19.2, C21.2, C23.2, R9.2, U9.4 (GND)
- net VIN: now also C21.1, C23.1, R11.2, U9.6 (VOUT); no longer U9.3 (VIN)
- net at U9.1 (FB): now also R11.1, R9.1
- net at U9.5 (SW): now also L1.2
Other:
- moved on the sheet: C17, C19, C21, C23, L1, R11, R9, U9
