File: LibreCube PCDU/My version/src/electrical/my_pcdu_v1.kicad_pcb (KiCad board)
At the start: 4 copper layers, 90.2 x 95.9 mm, 8 parts, among them M1 MountingHole, M2 MountingHole, M3 MountingHole, M4 MountingHole

Commit message: Updates
Parts:
- added BT1: Battery_Cell, Battery:BatteryHolder_Keystone_1042_1x18650, F.Cu at (231.8, 54.0)
- added BT2: Battery_Cell, Battery:BatteryHolder_Keystone_1042_1x18650, F.Cu at (231.8, 76.7)
- added C1: 10uF, Capacitor_SMD:C_0805_2012Metric, F.Cu at (243.3, 89.5)
- added C10: 0.22uF, Capacitor_SMD:C_0805_2012Metric, F.Cu at (247.7, 89.5)
- added C11: 10uF, Capacitor_SMD:C_0805_2012Metric, F.Cu at (247.7, 92.5)
- added C12: 10uF, Capacitor_SMD:C_0805_2012Metric, F.Cu at (247.7, 95.6)
- added C13: 0.1uF, Capacitor_SMD:C_0805_2012Metric, F.Cu at (247.7, 98.6)
- added C14: 0.1uF, Capacitor_SMD:C_0805_2012Metric, F.Cu at (247.7, 101.6)
- added C15: 0.1uF, Capacitor_SMD:C_0805_2012Metric, F.Cu at (247.7, 104.6)
- added C16: 0.1uF, Capacitor_SMD:C_0805_2012Metric, F.Cu at (247.7, 107.6)
- added C17: 10uF, Capacitor_SMD:C_0805_2012Metric, F.Cu at (252.2, 89.5)
- added C18: 10uF, Capacitor_SMD:C_0805_2012Metric, F.Cu at (252.2, 92.5)
- added C19: 2.2uF, Capacitor_SMD:C_0805_2012Metric, F.Cu at (252.2, 95.6)
- added C2: 10uF, Capacitor_SMD:C_0805_2012Metric, F.Cu at (243.3, 92.5)
- added C20: 2.2uF, Capacitor_SMD:C_0805_2012Metric, F.Cu at (252.2, 98.6)
- added C21: 220uF, Capacitor_Tantalum_SMD:CP_EIA-7343-31_Kemet-D, F.Cu at (236.1, 102.7)
- added C22: 220uF, Capacitor_Tantalum_SMD:CP_EIA-7343-31_Kemet-D, F.Cu at (236.1, 108.5)
- added C23: 0.1uF, Capacitor_SMD:C_0805_2012Metric, F.Cu at (252.2, 101.6)
- added C24: 0.1uF, Capacitor_SMD:C_0805_2012Metric, F.Cu at (252.2, 104.6)
- added C25: 0.1uF, Capacitor_SMD:C_0805_2012Metric, F.Cu at (252.2, 107.6)
- added C26: 0.1uF, Capacitor_SMD:C_0805_2012Metric, F.Cu at (256.6, 89.5)
- added C27: 0.1uF, Capacitor_SMD:C_0805_2012Metric, F.Cu at (256.6, 92.5)
- added C28: 0.1uF, Capacitor_SMD:C_0805_2012Metric, F.Cu at (256.6, 95.6)
- added C29: 0.1uF, Capacitor_SMD:C_0805_2012Metric, F.Cu at (256.6, 98.6)
- added C3: 2.2uF, Capacitor_SMD:C_0805_2012Metric, F.Cu at (243.3, 95.6)
- added C30: 0.1uF, Capacitor_SMD:C_0805_2012Metric, F.Cu at (256.6, 101.6)
- added C4: 2.2uF, Capacitor_SMD:C_0805_2012Metric, F.Cu at (243.3, 98.6)
- added C5: 220uF, Capacitor_Tantalum_SMD:CP_EIA-7343-31_Kemet-D, F.Cu at (236.1, 91.0)
- added C6: 220uF, Capacitor_Tantalum_SMD:CP_EIA-7343-31_Kemet-D, F.Cu at (236.1, 96.8)
- added C7: 10uF, Capacitor_SMD:C_0805_2012Metric, F.Cu at (243.3, 101.6)
- added C8: 10uF, Capacitor_SMD:C_0805_2012Metric, F.Cu at (243.3, 104.6)
- added C9: 0.22uF, Capacitor_SMD:C_0805_2012Metric, F.Cu at (243.3, 107.6)
- added D1: D_Schottky, Diode_SMD:D_SOD-123, F.Cu at (243.9, 110.8)
- added D10: D_Schottky, Diode_SMD:D_SOD-123, F.Cu at (249.7, 120.8)
- added D11: D_Schottky, Diode_SMD:D_SOD-123, F.Cu at (249.7, 124.2)
- added D12: D_Schottky, Diode_SMD:D_SOD-123, F.Cu at (249.7, 127.5)
- added D13: LED, Diode_SMD:D_0805_2012Metric, F.Cu at (260.7, 126.7)
- added D14: LED, Diode_SMD:D_0805_2012Metric, F.Cu at (260.7, 129.8)
- added D15: LED, Diode_SMD:D_0805_2012Metric, F.Cu at (260.7, 132.8)
- added D16: LED, Diode_SMD:D_0805_2012Metric, F.Cu at (265.1, 126.7)
- added D17: D_Schottky, Diode_SMD:D_SOD-123, F.Cu at (255.5, 110.8)
- added D18: D_Schottky, Diode_SMD:D_SOD-123, F.Cu at (255.5, 114.1)
- added D19: D_Schottky, Diode_SMD:D_SOD-123, F.Cu at (255.5, 117.5)
- added D2: D_Schottky, Diode_SMD:D_SOD-123, F.Cu at (243.9, 114.1)
- added D20: D_Schottky, Diode_SMD:D_SOD-123, F.Cu at (255.5, 120.8)
- added D21: LED, Diode_SMD:D_0805_2012Metric, F.Cu at (265.1, 129.8)
- added D22: LED, Diode_SMD:D_0805_2012Metric, F.Cu at (265.1, 132.8)
- added D23: LED, Diode_SMD:D_0805_2012Metric, F.Cu at (269.6, 126.7)
- added D24: LED, Diode_SMD:D_0805_2012Metric, F.Cu at (269.6, 129.8)
- added D25: LED, Diode_SMD:D_0805_2012Metric, F.Cu at (269.6, 132.8)
- added D3: D_Schottky, Diode_SMD:D_SOD-123, F.Cu at (243.9, 117.5)
- added D4: D_Schottky, Diode_SMD:D_SOD-123, F.Cu at (243.9, 120.8)
- added D5: D_Schottky, Diode_SMD:D_SOD-123, F.Cu at (243.9, 124.2)
- added D6: D_Schottky, Diode_SMD:D_SOD-123, F.Cu at (243.9, 127.5)
- added D7: D_Schottky, Diode_SMD:D_SOD-123, F.Cu at (249.7, 110.8)
- added D8: D_Schottky, Diode_SMD:D_SOD-123, F.Cu at (249.7, 114.1)
- added D9: D_Schottky, Diode_SMD:D_SOD-123, F.Cu at (249.7, 117.5)
- added J1: Conn_01x02, Connector_PinHeader_2.54mm:PinHeader_1x02_P2.54mm_Horizontal, F.Cu at (202.4, 90.4)
- added J2: Conn_01x02, Connector_PinHeader_2.54mm:PinHeader_1x02_P2.54mm_Horizontal, F.Cu at (202.4, 97.6)
- added J3: Conn_01x02, Connector_PinHeader_2.54mm:PinHeader_1x02_P2.54mm_Horizontal, F.Cu at (202.4, 104.8)
- added J4: Conn_01x02, Connector_PinHeader_2.54mm:PinHeader_1x02_P2.54mm_Horizontal, F.Cu at (202.4, 112.0)
- added J5: Conn_01x02, Connector_PinHeader_2.54mm:PinHeader_1x02_P2.54mm_Horizontal, F.Cu at (202.4, 119.2)
- added J6: Conn_01x02, Connector_PinHeader_2.54mm:PinHeader_1x02_P2.54mm_Horizontal, F.Cu at (202.4, 126.4)
- added J7: Conn_01x02, Connector_PinHeader_2.54mm:PinHeader_1x02_P2.54mm_Vertical, F.Cu at (269.9, 111.4)
- added L1: 6.8uH, Inductor_SMD:L_10.4x10.4_H4.8, F.Cu at (193.8, 94.0)
- added L2: 6.8uH, Inductor_SMD:L_10.4x10.4_H4.8, F.Cu at (193.8, 106.0)
- added L3: 6.8uH, Inductor_SMD:L_10.4x10.4_H4.8, F.Cu at (193.8, 117.9)
- added L4: 6.8uH, Inductor_SMD:L_10.4x10.4_H4.8, F.Cu at (193.8, 129.9)
- added R1: 0.1, Resistor_SMD:R_1206_3216Metric, F.Cu at (270.3, 117.9)
- added R10: 1.5k, Resistor_SMD:R_0805_2012Metric, F.Cu at (265.4, 89.5)
- added R11: 1M, Resistor_SMD:R_0805_2012Metric, F.Cu at (265.4, 92.5)
- added R12: 1M, Resistor_SMD:R_0805_2012Metric, F.Cu at (265.4, 95.4)
- added R13: 1M, Resistor_SMD:R_0805_2012Metric, F.Cu at (265.4, 98.4)
- added R14: 1M, Resistor_SMD:R_0805_2012Metric, F.Cu at (265.4, 101.3)
- added R15: 1M, Resistor_SMD:R_0805_2012Metric, F.Cu at (265.4, 104.3)
- added R16: 1.5k, Resistor_SMD:R_0805_2012Metric, F.Cu at (265.4, 107.2)
- added R17: 1.5k, Resistor_SMD:R_0805_2012Metric, F.Cu at (269.9, 89.5)
- added R18: 1.5k, Resistor_SMD:R_0805_2012Metric, F.Cu at (269.9, 92.5)
- added R19: 1.5k, Resistor_SMD:R_0805_2012Metric, F.Cu at (269.9, 95.4)
- added R2: 0.1, Resistor_SMD:R_1206_3216Metric, F.Cu at (270.3, 121.2)
- added R20: 1.5k, Resistor_SMD:R_0805_2012Metric, F.Cu at (269.9, 98.4)
- added R3: 309k, Resistor_SMD:R_0805_2012Metric, F.Cu at (261.0, 89.5)
- added R4: 110k, Resistor_SMD:R_0805_2012Metric, F.Cu at (261.0, 92.5)
- added R5: 309k, Resistor_SMD:R_0805_2012Metric, F.Cu at (261.0, 95.4)
- added R6: 110k, Resistor_SMD:R_0805_2012Metric, F.Cu at (261.0, 98.4)
- added R7: 1.5k, Resistor_SMD:R_0805_2012Metric, F.Cu at (261.0, 101.3)
- added R8: 1.5k, Resistor_SMD:R_0805_2012Metric, F.Cu at (261.0, 104.3)
- added R9: 1.5k, Resistor_SMD:R_0805_2012Metric, F.Cu at (261.0, 107.2)
- added U1: TPS61032, Package_SO:HTSSOP-16-1EP_4.4x5mm_P0.65mm_EP3x3mm, F.Cu at (226.7, 91.3)
- added U10: TPS2034, Package_SO:SO-8_3.9x4.9mm_P1.27mm, F.Cu at (217.7, 111.1)
- added U11: TPS2034, Package_SO:SO-8_3.9x4.9mm_P1.27mm, F.Cu at (217.7, 117.7)
- added U12: TPS2034, Package_SO:SO-8_3.9x4.9mm_P1.27mm, F.Cu at (217.7, 124.3)
- added U2: TPS61032, Package_SO:HTSSOP-16-1EP_4.4x5mm_P0.65mm_EP3x3mm, F.Cu at (226.7, 97.9)
- added U3: bq24002, Package_SO:HTSSOP-20-1EP_4.4x6.5mm_P0.65mm_EP2.85x4mm, F.Cu at (263.2, 113.1)
- added U4: bq24002, Package_SO:HTSSOP-20-1EP_4.4x6.5mm_P0.65mm_EP2.85x4mm, F.Cu at (263.2, 121.2)
- added U5: TPS2034, Package_SO:SO-8_3.9x4.9mm_P1.27mm, F.Cu at (217.7, 91.4)
- added U6: TPS2034, Package_SO:SO-8_3.9x4.9mm_P1.27mm, F.Cu at (217.7, 98.0)
- added U7: TPS61032, Package_SO:HTSSOP-16-1EP_4.4x5mm_P0.65mm_EP3x3mm, F.Cu at (226.7, 104.5)
- added U8: TPS61032, Package_SO:HTSSOP-16-1EP_4.4x5mm_P0.65mm_EP3x3mm, F.Cu at (226.7, 111.1)
- added U9: TPS2034, Package_SO:SO-8_3.9x4.9mm_P1.27mm, F.Cu at (217.7, 104.5)
Connections:
- net /CHARGE renamed CHARGE
- net /VBAT renamed +BATT
- H1 pad 33: /GND -> GND
- H1 pad 34: /GND -> GND
- H1 pad 45: /ENA_LCL_1 -> ENA_LCL_4
- H1 pad 46: /LCL_1 -> PWR_LCL_4
- H1 pad 47: /ENA_LCL_2 -> ENA_LCL_3
- H1 pad 48: /LCL_2 -> PWR_LCL_3
- H1 pad 49: /ENA_LCL_3 -> ENA_LCL_2
- H1 pad 50: /LCL_3 -> PWR_LCL_2
- H1 pad 51: /ENA_LCL_4 -> ENA_LCL_1
- H1 pad 52: /LCL_4 -> PWR_LCL_1
- H2 pad 25: /5V -> +5V
- H2 pad 26: /5V -> +5V
- H2 pad 29: /GND -> GND
- H2 pad 30: /GND -> GND
- H2 pad 31: /GND -> GND
- H2 pad 32: /GND -> GND
- H2 pad 33: /ENA_LCL_5 -> unconnected-(H2-Pin_33-Pad33)
- H2 pad 34: /LCL_5 -> unconnected-(H2-Pin_34-Pad34)
- H2 pad 35: /ENA_LCL_6 -> unconnected-(H2-Pin_35-Pad35)
- H2 pad 36: /LCL_6 -> unconnected-(H2-Pin_36-Pad36)
- H2 pad 37: /ENA_LCL_7 -> S2
- H2 pad 38: /LCL_7 -> S2
- H2 pad 39: /ENA_LCL_8 -> S2
- H2 pad 40: /LCL_8 -> S2
- H2 pad 41: unconnected-(H2-Pin_41-Pad41) -> GND
- H2 pad 42: unconnected-(H2-Pin_42-Pad42) -> GND
- H2 pad 43: unconnected-(H2-Pin_43-Pad43) -> GND
- H2 pad 44: unconnected-(H2-Pin_44-Pad44) -> GND
Routing:
- added copper zone on In1.Cu, net GND
- added copper zone on In2.Cu, net GND
- removed copper zone on In1.Cu, net /GND
- removed copper zone on In2.Cu, net /GND

Commit message: Updates
Parts:
- removed the U4 at (263.2, 121.2)
- added U8: bq24002, Package_SO:HTSSOP-20-1EP_4.4x6.5mm_P0.65mm_EP2.85x4mm, F.Cu at (278.6, 121.0)
- moved BT2 104.6 mm to (127.3, 74.9)
- renumbered C23 to C1, C2 to C10, C3 to C11, C4 to C12, C5 to C13, C6 to C14, C7 to C15, C8 to C16, C9 to C17, C10 to C18, C11 to C19, C24 to C2, C12 to C20, C13 to C21, C14 to C22, C15 to C23, C16 to C24, C17 to C25, C18 to C26, C19 to C27, C20 to C28, C21 to C29, C25 to C3, C22 to C30, C26 to C4, C27 to C5, C28 to C6, C29 to C7, C30 to C8, C1 to C9, D21 to D13, D22 to D14, D23 to D15, D24 to D16, D13 to D17, D14 to D18, D15 to D19, D16 to D20, D25 to D21, D17 to D22, D18 to D23, D19 to D24, D20 to D25, R12 to R1, R4 to R10, R5 to R11, R6 to R12, R18 to R13, R19 to R14, R7 to R15, R8 to R16, R9 to R17, R10 to R18, R20 to R19, R13 to R2, R11 to R20, R14 to R3, R15 to R4, R16 to R5, R1 to R6, R2 to R7, R17 to R8, R3 to R9, U9 to U1, U6 to U10, U7 to U11, U8 to U12, U10 to U2, U11 to U3, U12 to U4, U1 to U5, U2 to U6, U3 to U7, U5 to U9
Connections:
- H1 pad 1: /CAN_A_L -> unconnected-(H1-Pin_1-Pad1)
- H1 pad 13: /UART_C_TX -> unconnected-(H1-Pin_13-Pad13)
- H1 pad 15: /UART_C_RX -> unconnected-(H1-Pin_15-Pad15)
- H1 pad 2: /CAN_B_L -> unconnected-(H1-Pin_2-Pad2)
- H1 pad 22: /UART_D_TX -> unconnected-(H1-Pin_22-Pad22)
- H1 pad 24: /UART_D_RX -> unconnected-(H1-Pin_24-Pad24)
- H1 pad 25: /5V -> +5V
- H1 pad 26: /5V -> +5V
- H1 pad 3: /CAN_A_H -> unconnected-(H1-Pin_3-Pad3)
- H1 pad 4: /CAN_B_H -> unconnected-(H1-Pin_4-Pad4)
- H1 pad 5: /UART_A_TX -> unconnected-(H1-Pin_5-Pad5)
- H1 pad 6: /UART_B_TX -> unconnected-(H1-Pin_6-Pad6)
- H1 pad 7: /UART_A_RX -> unconnected-(H1-Pin_7-Pad7)
- H1 pad 8: /UART_B_RX -> unconnected-(H1-Pin_8-Pad8)
- U7 pad 21: (no net) -> unconnected-(U7-NC-Pad21)

Commit message: Uploaded PCDUv2
Connections:
- D13 pad 2: PWR_LCL_1 -> PWR_LCL_4
- D14 pad 2: PWR_LCL_2 -> PWR_LCL_3
- D15 pad 2: PWR_LCL_3 -> PWR_LCL_2
- D16 pad 2: PWR_LCL_4 -> PWR_LCL_1
- H1 pad 45: ENA_LCL_4 -> ENA_LCL_1
- H1 pad 46: PWR_LCL_4 -> PWR_LCL_1
- H1 pad 47: ENA_LCL_3 -> ENA_LCL_2
- H1 pad 48: PWR_LCL_3 -> PWR_LCL_2
- H1 pad 49: ENA_LCL_2 -> ENA_LCL_3
- H1 pad 50: PWR_LCL_2 -> PWR_LCL_3
- H1 pad 51: ENA_LCL_1 -> ENA_LCL_4
- H1 pad 52: PWR_LCL_1 -> PWR_LCL_4
Changed lines of the file:
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@@
 			(layers "*.Cu" "*.Mask")
 			(remove_unused_layers no)
-			(net 107 "ENA_LCL_4")
+			(net 106 "ENA_LCL_1")
 			(pinfunction "Pin_45")
 			(pintype "passive")
@@
 			(layers "*.Cu" "*.Mask")
 			(remove_unused_layers no)
-			(net 78 "PWR_LCL_4")
+			(net 47 "PWR_LCL_1")
 			(pinfunction "Pin_46")
 			(pintype "passive")
@@
 			(layers "*.Cu" "*.Mask")
 			(remove_unused_layers no)
-			(net 105 "ENA_LCL_3")
+			(net 104 "ENA_LCL_2")
 			(pinfunction "Pin_47")
 			(pintype "passive")
@@
 			(layers "*.Cu" "*.Mask")
 			(remove_unused_layers no)
-			(net 77 "PWR_LCL_3")
+			(net 48 "PWR_LCL_2")
 			(pinfunction "Pin_48")
 			(pintype "passive")
@@
 			(layers "*.Cu" "*.Mask")
 			(remove_unused_layers no)
-			(net 104 "ENA_LCL_2")
+			(net 105 "ENA_LCL_3")
 			(pinfunction "Pin_49")
 			(pintype "passive")
@@
 			(layers "*.Cu" "*.Mask")
 			(remove_unused_layers no)
-			(net 48 "PWR_LCL_2")
+			(net 77 "PWR_LCL_3")
 			(pinfunction "Pin_50")
 			(pintype "passive")
@@
 			(layers "*.Cu" "*.Mask")
 			(remove_unused_layers no)
-			(net 106 "ENA_LCL_1")
+			(net 107 "ENA_LCL_4")
 			(pinfunction "Pin_51")
 			(pintype "passive")
@@
 			(layers "*.Cu" "*.Mask")
 			(remove_unused_layers no)
-			(net 47 "PWR_LCL_1")
+			(net 78 "PWR_LCL_4")
 			(pinfunction "Pin_52")
 			(pintype "passive")
@@
 			(layers "F.Cu" "F.Paste" "F.Mask")
 			(roundrect_rratio 0.25)
-			(net 47 "PWR_LCL_1")
+			(net 78 "PWR_LCL_4")
 			(pinfunction "A")
 			(pintype "passive")
@@
 			(layers "F.Cu" "F.Paste" "F.Mask")
 			(roundrect_rratio 0.25)
-			(net 78 "PWR_LCL_4")
+			(net 47 "PWR_LCL_1")
 			(pinfunction "A")
 			(pintype "passive")
@@
 			(layers "F.Cu" "F.Paste" "F.Mask")
 			(roundrect_rratio 0.25)
-			(net 48 "PWR_LCL_2")
+			(net 77 "PWR_LCL_3")
 			(pinfunction "A")
 			(pintype "passive")
@@
 			(layers "F.Cu" "F.Paste" "F.Mask")
 			(roundrect_rratio 0.25)
-			(net 77 "PWR_LCL_3")
+			(net 48 "PWR_LCL_2")
 			(pinfunction "A")
 			(pintype "passive")

Commit message: More updates
Parts:
- added C31: 0.1uF, Capacitor_SMD:C_0805_2012Metric, F.Cu at (224.3, 136.6)
- added C32: 0.1uF, Capacitor_SMD:C_0805_2012Metric, F.Cu at (224.3, 139.6)
- added C33: 0.1uF, Capacitor_SMD:C_0805_2012Metric, F.Cu at (224.3, 142.6)
- added C34: 0.1uF, Capacitor_SMD:C_0805_2012Metric, F.Cu at (224.3, 145.7)
- added C35: 0.1uF, Capacitor_SMD:C_0805_2012Metric, F.Cu at (224.3, 148.7)
- added C36: 0.1uF, Capacitor_SMD:C_0805_2012Metric, F.Cu at (224.3, 151.7)
- added C37: 0.1uF, Capacitor_SMD:C_0805_2012Metric, F.Cu at (224.3, 154.7)
- added C38: 0.1uF, Capacitor_SMD:C_0805_2012Metric, F.Cu at (224.3, 157.7)
- added J8: USB_C_Receptacle_PowerOnly_6P, Connector_USB:USB_C_Receptacle_GCT_USB4125-xx-x-0190_6P_TopMnt_Horizontal, F.Cu at (232.4, 157.7)
- added R21: 1M, Resistor_SMD:R_0805_2012Metric, F.Cu at (228.7, 142.5)
- added R22: 1M, Resistor_SMD:R_0805_2012Metric, F.Cu at (228.7, 145.4)
- added R23: 1M, Resistor_SMD:R_0805_2012Metric, F.Cu at (228.7, 148.4)
- added R24: 1M, Resistor_SMD:R_0805_2012Metric, F.Cu at (228.7, 151.3)
- added R5: 5.1k, Resistor_SMD:R_0805_2012Metric, F.Cu at (228.7, 136.6)
- added R8: 5.1k, Resistor_SMD:R_0805_2012Metric, F.Cu at (228.7, 139.5)
- added U13: TPS2034, Package_SO:SO-8_3.9x4.9mm_P1.27mm, F.Cu at (217.8, 138.5)
- added U14: TPS2034, Package_SO:SO-8_3.9x4.9mm_P1.27mm, F.Cu at (217.8, 145.1)
- added U15: TPS2034, Package_SO:SO-8_3.9x4.9mm_P1.27mm, F.Cu at (217.8, 151.6)
- added U16: TPS2034, Package_SO:SO-8_3.9x4.9mm_P1.27mm, F.Cu at (217.8, 158.2)
Connections:
- H2 pad 33: unconnected-(H2-Pin_33-Pad33) -> ENA_LCL_5
- H2 pad 34: unconnected-(H2-Pin_34-Pad34) -> PWR_LCL_5
- H2 pad 35: unconnected-(H2-Pin_35-Pad35) -> ENA_LCL_6
- H2 pad 36: unconnected-(H2-Pin_36-Pad36) -> PWR_LCL_6
- H2 pad 37: S2 -> ENA_LCL_7
- H2 pad 38: S2 -> PWR_LCL_7
- H2 pad 39: S2 -> ENA_LCL_8
- H2 pad 40: S2 -> PWR_LCL_8
- H2 pad 41: GND -> unconnected-(H2-Pin_41-Pad41)
- H2 pad 42: GND -> unconnected-(H2-Pin_42-Pad42)
- H2 pad 43: GND -> unconnected-(H2-Pin_43-Pad43)
- H2 pad 44: GND -> unconnected-(H2-Pin_44-Pad44)
- H2 pad 49: unconnected-(H2-Pin_49-Pad49) -> KS_OPEN
- H2 pad 50: unconnected-(H2-Pin_50-Pad50) -> GND
- H2 pad 51: unconnected-(H2-Pin_51-Pad51) -> KS_OPEN
- H2 pad 52: unconnected-(H2-Pin_52-Pad52) -> GND
- J7 pad 1: S2 -> KS_OPEN
- R20 pad 2: S2 -> KS_OPEN
- U10 pad 4: S2 -> KS_OPEN
- U9 pad 4: S2 -> KS_OPEN

Commit message: PCDU updates
Parts:
- removed C29, C30: 220uF, Capacitor_Tantalum_SMD:CP_EIA-7343-31_Kemet-D
- removed D17, D18, D19, D20: LED, Diode_SMD:D_0805_2012Metric
- removed L3, L4: 6.8uH, Inductor_SMD:L_10.4x10.4_H4.8
- removed the R5 at (265.4, 107.2)
- removed the R8 at (269.9, 89.5)
- removed U11, U12: TPS61032, Package_SO:HTSSOP-16-1EP_4.4x5mm_P0.65mm_EP3x3mm
- removed U8: bq24002, Package_SO:HTSSOP-20-1EP_4.4x6.5mm_P0.65mm_EP2.85x4mm
- added R25: 100k, Resistor_SMD:R_0805_2012Metric_Pad1.20x1.40mm_HandSolder, F.Cu at (63.5, 109.1)
- added R26: 100k, Resistor_SMD:R_0805_2012Metric_Pad1.20x1.40mm_HandSolder, F.Cu at (63.5, 112.1)
- added R27: 1k5, Resistor_SMD:R_0805_2012Metric_Pad1.20x1.40mm_HandSolder, F.Cu at (63.5, 115.0)
- added R28: 1k5, Resistor_SMD:R_0805_2012Metric_Pad1.20x1.40mm_HandSolder, F.Cu at (68.2, 103.2)
- added R29: 100k, Resistor_SMD:R_0805_2012Metric_Pad1.20x1.40mm_HandSolder, F.Cu at (68.2, 106.2)
- added R30: 10k, Resistor_SMD:R_0805_2012Metric_Pad1.20x1.40mm_HandSolder, F.Cu at (68.2, 109.1)
- added R31: 820Ω, Resistor_SMD:R_0805_2012Metric_Pad1.20x1.40mm_HandSolder, F.Cu at (68.2, 112.1)
- added R32: 37k4, Resistor_SMD:R_0805_2012Metric_Pad1.20x1.40mm_HandSolder, F.Cu at (68.2, 115.0)
- added U17: TPS61023DRLR, TPS61023DRLR:DRL0006A, F.Cu at (113.3, 109.5)
- added U19: TPS61232DRCR, TPS61232DRCR:VREG_TPS61232DRCR, F.Cu at (94.0, 108.3)
- added U20: TPS61232DRCR, TPS61232DRCR:VREG_TPS61232DRCR, F.Cu at (94.0, 113.3)
- C10, C19, C20, C9: footprint Capacitor_SMD:C_0805_2012Metric -> Capacitor_SMD:C_0805_2012Metric_Pad1.18x1.45mm_HandSolder
- C11, C12, C27, C28: value 2.2uF -> 10uF; footprint Capacitor_SMD:C_0805_2012Metric -> Capacitor_SMD:C_0805_2012Metric_Pad1.18x1.45mm_HandSolder
- C13, C14: value 220uF -> 22uF; footprint Capacitor_Tantalum_SMD:CP_EIA-7343-31_Kemet-D -> Capacitor_SMD:C_0805_2012Metric_Pad1.18x1.45mm_HandSolder
- C15, C16: value 10uF -> 22uF; footprint Capacitor_SMD:C_0805_2012Metric -> Capacitor_SMD:C_0805_2012Metric_Pad1.18x1.45mm_HandSolder
- C17, C18: value 0.22uF -> 10u; footprint Capacitor_SMD:C_0805_2012Metric -> Capacitor_SMD:C_1206_3216Metric_Pad1.33x1.80mm_HandSolder
- C25, C26: value 10uF -> 10u; footprint Capacitor_SMD:C_0805_2012Metric -> Capacitor_SMD:C_1206_3216Metric_Pad1.33x1.80mm_HandSolder
- D13, D15: value LED -> Red; footprint Diode_SMD:D_0805_2012Metric -> LED_SMD:LED_0805_2012Metric_Pad1.15x1.40mm_HandSolder
- D14, D16: value LED -> Green; footprint Diode_SMD:D_0805_2012Metric -> LED_SMD:LED_0805_2012Metric_Pad1.15x1.40mm_HandSolder
- L1, L2: value 6.8uH -> 1uH; footprint Inductor_SMD:L_10.4x10.4_H4.8 -> Inductor_SMD:L_Coilcraft_XxL4040
- R10: value 110k -> 750k; footprint Resistor_SMD:R_0805_2012Metric -> Resistor_SMD:R_0805_2012Metric_Pad1.20x1.40mm_HandSolder
- R11: value 309k -> 10k; footprint Resistor_SMD:R_0805_2012Metric -> Resistor_SMD:R_0805_2012Metric_Pad1.20x1.40mm_HandSolder
- R12: value 110k -> 100k; footprint Resistor_SMD:R_0805_2012Metric -> Resistor_SMD:R_0805_2012Metric_Pad1.20x1.40mm_HandSolder
- R13, R18: value 1.5k -> 100k; footprint Resistor_SMD:R_0805_2012Metric -> Resistor_SMD:R_0805_2012Metric_Pad1.20x1.40mm_HandSolder
- R14, R15: value 1.5k -> 1k5; footprint Resistor_SMD:R_0805_2012Metric -> Resistor_SMD:R_0805_2012Metric_Pad1.20x1.40mm_HandSolder
- R16: value 1.5k -> 820Ω; footprint Resistor_SMD:R_0805_2012Metric -> Resistor_SMD:R_0805_2012Metric_Pad1.20x1.40mm_HandSolder
- R17: value 1.5k -> 37k4; footprint Resistor_SMD:R_0805_2012Metric -> Resistor_SMD:R_0805_2012Metric_Pad1.20x1.40mm_HandSolder
- R6: value 0.1 -> 750k; footprint Resistor_SMD:R_1206_3216Metric -> Resistor_SMD:R_0805_2012Metric_Pad1.20x1.40mm_HandSolder
- R7: value 0.1 -> 100k; footprint Resistor_SMD:R_1206_3216Metric -> Resistor_SMD:R_0805_2012Metric_Pad1.20x1.40mm_HandSolder
- R9: value 309k -> 100k; footprint Resistor_SMD:R_0805_2012Metric -> Resistor_SMD:R_0805_2012Metric_Pad1.20x1.40mm_HandSolder
- U5: value TPS61032 -> BQ24032ARHLRG4; footprint Package_SO:HTSSOP-16-1EP_4.4x5mm_P0.65mm_EP3x3mm -> BQ24032ARHLRG4:IC_MSP430FR2522IRHLR
- U6: value TPS61032 -> TPS61023DRLR; footprint Package_SO:HTSSOP-16-1EP_4.4x5mm_P0.65mm_EP3x3mm -> TPS61023DRLR:DRL0006A
- U7: value bq24002 -> BQ24032ARHLRG4; footprint Package_SO:HTSSOP-20-1EP_4.4x6.5mm_P0.65mm_EP2.85x4mm -> BQ24032ARHLRG4:IC_MSP430FR2522IRHLR
- moved R7 216.9 mm to (54.0, 106.2)
- moved R6 216.9 mm to (54.0, 103.2)
- moved R13 211.6 mm to (58.7, 106.2)
- moved R14 211.6 mm to (58.7, 109.1)
- moved R10 208.0 mm to (54.0, 112.1)
- moved R11 208.0 mm to (54.0, 115.0)
- moved R9 208.0 mm to (54.0, 109.1)
- moved R18 202.7 mm to (63.5, 106.2)
- moved R15 202.6 mm to (58.7, 112.1)
- moved R16 202.6 mm to (58.7, 115.0)
- moved R12 202.4 mm to (58.7, 103.2)
- moved R17 197.6 mm to (63.5, 103.2)
- moved C10 191.4 mm to (54.0, 121.0)
- moved C11 191.4 mm to (54.0, 124.0)
- moved C12 191.4 mm to (54.0, 127.0)
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Connections:
- C11 pad 1: Net-(D22-A) -> CHARGE
- C12 pad 1: Net-(D22-A) -> CHARGE
- C17 pad 1: Net-(U7-CR) -> Net-(D22-A)
- C18 pad 1: Net-(U8-CR) -> Net-(D22-A)
- C19 pad 1: +BATT -> Net-(D24-A)
- C23 pad 1: Net-(U11-EN) -> Net-(C23-Pad1)
- C24 pad 1: Net-(U11-EN) -> Net-(C23-Pad1)
- C25 pad 1: Net-(U11-EN) -> Net-(D22-A)
- C26 pad 1: Net-(U11-EN) -> Net-(D22-A)
- C27 pad 1: +5V -> +BATT
- C28 pad 1: +5V -> Net-(D24-A)
- D13 pad 2: PWR_LCL_4 -> Net-(D13-A)
- D14 pad 2: PWR_LCL_3 -> Net-(D14-A)
- D15 pad 2: PWR_LCL_2 -> Net-(D15-A)
- D16 pad 2: PWR_LCL_1 -> Net-(D16-A)
- D24 pad 2: +BATT -> Net-(D24-A)
- D25 pad 2: +BATT -> Net-(D24-A)
- L1 pad 1: Net-(L1-Pad1) -> CHARGE
- L1 pad 2: CHARGE -> Net-(U17-SW)
- L2 pad 1: Net-(L2-Pad1) -> CHARGE
- L2 pad 2: CHARGE -> Net-(U6-SW)
- R10 pad 1: Net-(U7-APG/THERM) -> Net-(U6-FB)
- R10 pad 2: GND -> Net-(D22-A)
- R11 pad 1: Net-(D22-A) -> Net-(U7-TS)
- R11 pad 2: Net-(U8-APG/THERM) -> GND
- R12 pad 1: Net-(U8-APG/THERM) -> Net-(D22-A)
- R12 pad 2: GND -> Net-(U7-PSEL)
- R13 pad 1: Net-(D15-K) -> Net-(D22-A)
- R13 pad 2: GND -> Net-(U7-CE)
- R14 pad 1: Net-(D16-K) -> Net-(D22-A)
- R14 pad 2: GND -> Net-(D13-A)
- R15 pad 2: Net-(D17-A) -> Net-(D14-A)
- R16 pad 1: Net-(D22-A) -> Net-(U7-ISET1)
- R16 pad 2: Net-(D18-A) -> GND
- R17 pad 1: Net-(D22-A) -> Net-(U7-DPPM)
- R17 pad 2: Net-(D19-A) -> GND
- R18 pad 2: Net-(D20-A) -> Net-(U7-ISET2)
- R6 pad 1: Net-(U7-ISNS) -> Net-(U17-FB)
- R7 pad 1: Net-(U8-ISNS) -> Net-(U17-FB)
- R7 pad 2: Net-(D22-A) -> GND
- R9 pad 1: Net-(D22-A) -> Net-(U6-FB)
- R9 pad 2: Net-(U7-APG/THERM) -> GND
- U10 pad 6: Net-(U11-EN) -> Net-(C23-Pad1)
- U10 pad 7: Net-(U11-EN) -> Net-(C23-Pad1)
- U10 pad 8: Net-(U11-EN) -> Net-(C23-Pad1)
- U5 pad 1: Net-(L1-Pad1) -> Net-(U5-LDO)
- U5 pad 10: unconnected-(U5-LBO-Pad10) -> Net-(U5-ISET1)
- U5 pad 12: unconnected-(U5-FB-Pad12) -> Net-(U5-TS)
- U5 pad 13: Net-(D22-A) -> Net-(U5-DPPM)
- U5 pad 14: Net-(D22-A) -> Net-(U5-LDO)
- U5 pad 15: Net-(D22-A) -> Net-(D24-A)
- U5 pad 16: unconnected-(U5-NC-Pad16) -> Net-(D24-A)
- U5 pad 17: GND -> Net-(D24-A)
- U5 pad 2: Net-(L1-Pad1) -> Net-(D15-K)
- U5 pad 3: GND -> Net-(D16-K)
- U5 pad 4: GND -> Net-(D22-A)
- U5 pad 5: GND -> +BATT
- U5 pad 6: CHARGE -> +BATT
- U5 pad 7: GND -> Net-(U5-ISET2)
- U5 pad 8: GND -> Net-(U5-PSEL)
- U5 pad 9: CHARGE -> Net-(U5-CE)
- U6 pad 1: Net-(L2-Pad1) -> Net-(U6-FB)
- U6 pad 2: Net-(L2-Pad1) -> CHARGE
- U6 pad 3: GND -> CHARGE
- U6 pad 5: GND -> Net-(U6-SW)
- U6 pad 6: CHARGE -> Net-(D22-A)
- U7 pad 1: unconnected-(U7-NC-Pad1) -> Net-(U7-LDO)
- U7 pad 10: GND -> Net-(U7-ISET1)
- U7 pad 11: unconnected-(U7-NC-Pad11) -> GND
- U7 pad 12: Net-(U7-CR) -> Net-(U7-TS)
- U7 pad 13: GND -> Net-(U7-DPPM)
- U7 pad 14: Net-(D19-K) -> Net-(U7-LDO)
- U7 pad 15: Net-(D17-K) -> Net-(D24-A)
- U7 pad 16: GND -> Net-(D24-A)
- U7 pad 17: +BATT -> Net-(D24-A)
- U7 pad 18: +BATT -> unconnected-(U7-~{ACPG}-Pad18)
- U7 pad 19: +BATT -> unconnected-(U7-~{USBPG}-Pad19)
- U7 pad 2: Net-(U7-ISNS) -> Net-(D13-K)
- U7 pad 21: unconnected-(U7-NC-Pad21) -> (no net)
- U7 pad 3: Net-(U7-ISNS) -> Net-(D14-K)
- U7 pad 5: Net-(U7-ISNS) -> +BATT
- U7 pad 6: unconnected-(U7-NC-Pad6) -> +BATT
- U7 pad 7: Net-(U7-APG/THERM) -> Net-(U7-ISET2)
- U7 pad 8: Net-(D22-A) -> Net-(U7-PSEL)
- U7 pad 9: Net-(D22-A) -> Net-(U7-CE)
- U9 pad 6: Net-(U11-EN) -> Net-(C23-Pad1)
- U9 pad 7: Net-(U11-EN) -> Net-(C23-Pad1)
- U9 pad 8: Net-(U11-EN) -> Net-(C23-Pad1)

Commit message: PCB Layout
Parts:
- removed U20: TPS61232DRCR, TPS61232DRCR:VREG_TPS61232DRCR
- removed the U5 at (68.8, 120.2)
- added C37: 22uF, Capacitor_SMD:C_0805_2012Metric_Pad1.18x1.45mm_HandSolder, F.Cu at (49.3, 73.9)
- added C38: 22uF, Capacitor_SMD:C_0805_2012Metric_Pad1.18x1.45mm_HandSolder, F.Cu at (54.1, 64.8)
- added C39: 10nF, Capacitor_SMD:C_0805_2012Metric_Pad1.18x1.45mm_HandSolder, F.Cu at (49.3, 76.9)
- added C40: 10nF, Capacitor_SMD:C_0805_2012Metric_Pad1.18x1.45mm_HandSolder, F.Cu at (54.1, 67.9)
- added C41: 22uF, Capacitor_SMD:C_0805_2012Metric_Pad1.18x1.45mm_HandSolder, F.Cu at (49.3, 64.8)
- added C42: 22uF, Capacitor_SMD:C_0805_2012Metric_Pad1.18x1.45mm_HandSolder, F.Cu at (54.1, 70.9)
- added C43: 22uF, Capacitor_SMD:C_0805_2012Metric_Pad1.18x1.45mm_HandSolder, F.Cu at (49.3, 67.9)
- added C44: 22uF, Capacitor_SMD:C_0805_2012Metric_Pad1.18x1.45mm_HandSolder, F.Cu at (54.1, 73.9)
- added C45: 22uF, Capacitor_SMD:C_0805_2012Metric_Pad1.18x1.45mm_HandSolder, F.Cu at (49.3, 70.9)
- added C46: 22uF, Capacitor_SMD:C_0805_2012Metric_Pad1.18x1.45mm_HandSolder, F.Cu at (54.1, 76.9)
- added L3: 1uH, Inductor_SMD:L_Coilcraft_XAL4040-XXX, F.Cu at (33.4, 111.0)
- added L4: 1uH, Inductor_SMD:L_Coilcraft_XAL4040-XXX, F.Cu at (33.4, 116.9)
- added U12: BQ24032ARHLRG4, BQ24032ARHLRG4:IC_MSP430FR2522IRHLR, F.Cu at (64.1, 133.3)
- added U16: TPS61232DRCR, TPS61232DRCR:VREG_TPS61232DRCR, F.Cu at (59.5, 77.0)
- L1, L2: footprint Inductor_SMD:L_Coilcraft_XxL4040 -> Inductor_SMD:L_Coilcraft_XAL4040-XXX
- moved D1 150.1 mm to (93.9, 114.9), turned to -90 degrees
- moved D2 147.6 mm to (96.4, 114.9), turned to -90 degrees
- moved D3 142.8 mm to (101.2, 114.9), turned to -90 degrees
- moved D4 140.3 mm to (103.8, 114.9), turned to -90 degrees
- moved D5 135.7 mm to (108.6, 114.9), turned to -90 degrees
- moved D7 133.9 mm to (116.0, 114.9), turned to -90 degrees
- moved D6 133.4 mm to (111.1, 114.9), turned to -90 degrees
- moved D8 131.3 mm to (118.5, 114.9), turned to -90 degrees
- moved D9 126.5 mm to (123.3, 114.9), turned to -90 degrees
- moved D10 124.0 mm to (125.9, 114.9), turned to -90 degrees
- moved D11 119.4 mm to (130.7, 114.9), turned to -90 degrees
- moved D12 117.2 mm to (133.2, 114.9), turned to -90 degrees
- moved J1 109.9 mm to (96.4, 119.4), turned to -90 degrees
- moved BT1 106.9 mm to (127.6, 77.8), turned to 180 degrees
- moved J2 101.0 mm to (103.8, 119.4), turned to -90 degrees
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- renumbered C6 to C10, C7 to C11, C8 to C12, C35 to C13, C36 to C14, C37 to C15, C38 to C16, C9 to C17, C11 to C18, C10 to C19, C12 to C20, C13 to C21, C15 to C22, C14 to C23, C16 to C24, C17 to C25, C25 to C26, C18 to C27, C26 to C28, C20 to C29, C27 to C30, C19 to C31, C28 to C32, C21 to C33, C22 to C34, C23 to C35, C24 to C36, C31 to C5, C32 to C6, C33 to C7, C34 to C8, C5 to C9, D22 to D17, D23 to D18, D21 to D19, D24 to D20, D25 to D21, R9 to R10, R6 to R11, R10 to R12, R12 to R13, R13 to R14, R14 to R15, R15 to R16, R18 to R17, R25 to R18, R26 to R19, R27 to R20, R28 to R21, R29 to R22, R11 to R23, R30 to R24, R16 to R25, R31 to R26, R17 to R27, R32 to R28, R19 to R29, R20 to R30, R5 to R31, R8 to R32, R21 to R5, R22 to R6, R23 to R7, R24 to R8, R7 to R9, U6 to U10, U7 to U11, U9 to U13, U10 to U14, U19 to U15, U13 to U5, U14 to U6, U15 to U7, U16 to U8, U17 to U9
Connections:
- C35 pad 1: Net-(C23-Pad1) -> Net-(U15-EN)
- C36 pad 1: Net-(C23-Pad1) -> Net-(U15-EN)
- U11 pad 21: (no net) -> GND
- U13 pad 6: Net-(C23-Pad1) -> Net-(U15-EN)
- U13 pad 7: Net-(C23-Pad1) -> Net-(U15-EN)
- U13 pad 8: Net-(C23-Pad1) -> Net-(U15-EN)
- U14 pad 6: Net-(C23-Pad1) -> Net-(U15-EN)
- U14 pad 7: Net-(C23-Pad1) -> Net-(U15-EN)
- U14 pad 8: Net-(C23-Pad1) -> Net-(U15-EN)
- U15 pad 10: unconnected-(U19-VIN-Pad10) -> Net-(U15-EN)
- U15 pad 11: Net-(U19-GND-Pad11) -> GND
- U15 pad 11_1: Net-(U19-GND-Pad11) -> GND
- U15 pad 11_2: Net-(U19-GND-Pad11) -> GND
- U15 pad 11_3: Net-(U19-GND-Pad11) -> GND
- U15 pad 11_4: Net-(U19-GND-Pad11) -> GND
- U15 pad 3: Net-(U19-VOUT-Pad3) -> +5V
- U15 pad 4: Net-(U19-VOUT-Pad3) -> +5V
- U15 pad 6: unconnected-(U19-SS-Pad6) -> Net-(U15-SS)
- U15 pad 7: unconnected-(U19-FB-Pad7) -> +5V
- U15 pad 9: unconnected-(U19-EN-Pad9) -> Net-(U15-EN)

Commit message: Updates
Parts:
- C17, C18, C19, C20, C21, C22, C23, C24, C25, C26, C27, C28, C29, C30, C31, C32, C33, C34, C35, C36, C37, C38, C39, C40, C41, C42, C43, C44, C45, C46, D13, D14, D15, D16, D17, D18, D20, D21, L1, L2, L3, L4, R10, R11, R12, R13, R14, R15, R16, R17, R18, R19, R20, R21, R22, R23, R24, R25, R26, R27, R28, R30, R9, U10, U11, U12, U13, U14, U15, U16, U9: moved to B.Cu
- moved R30 150.8 mm to (114.9, 83.9), turned to 90 degrees
- moved D17 143.5 mm to (112.9, 95.1), turned to -90 degrees
- moved C36 142.1 mm to (108.8, 77.3)
- moved D18 141.4 mm to (115.4, 95.1), turned to -90 degrees
- moved C34 139.6 mm to (108.8, 86.9)
- moved C35 127.2 mm to (123.4, 77.3)
- moved D21 125.9 mm to (136.5, 79.8)
- moved C33 124.8 mm to (123.4, 87.0)
- moved D20 124.1 mm to (136.5, 82.4)
- moved C32 113.4 mm to (149.0, 67.1)
- moved U14 111.8 mm to (107.1, 82.1), turned to 90 degrees
- moved C30 104.8 mm to (145.3, 75.0), turned to 180 degrees
- moved R16 104.4 mm to (152.0, 108.5)
- moved R15 104.4 mm to (152.0, 110.8)
- moved R20 104.3 mm to (152.0, 83.9)
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Connections:
- net Net-(D17-A) renamed /VIN
- net Net-(D20-A) renamed /VOUT
Routing:
- net Net-(U11-LDO): track 0.00 -> 9.55 mm, vias 0 -> 2
- net Net-(U12-DPPM): track 0.00 -> 4.63 mm
- net Net-(U11-DPPM): track 0.00 -> 4.59 mm
- net Net-(U12-TS): track 0.00 -> 2.14 mm
- net Net-(U11-TS): track 0.00 -> 2.09 mm
- net Net-(U11-ISET1): track 0.00 -> 2.02 mm
- net Net-(U12-ISET1): track 0.00 -> 1.88 mm
- added copper zone on B.Cu, net +5V
- added copper zone on B.Cu, net /Semi_Regulated_Bus
- added copper zone on B.Cu, net Net-(U10-SW)
- removed copper zone on In1.Cu, net GND
- removed copper zone on In2.Cu, net GND
