File: LibreCube PCDU/My version/src/electrical/my_pcdu_v1.kicad_pcb (KiCad board)
At the start: 4 copper layers, 90.2 x 95.9 mm, 137 parts, among them J1 Conn_01x02, J2 Conn_01x02, J3 Conn_01x02, J4 Conn_01x02, J5 Conn_01x02, J6 Conn_01x02, J7 Conn_01x02, J8 USB_C_Receptacle_PowerOnly_6P, M1 MountingHole, M2 MountingHole, M3 MountingHole, M4 MountingHole, U1 TPS2034, U10 TPS61023DRLR, U11 BQ24032ARHLRG4, U12 BQ24032ARHLRG4, U13 TPS2034, U14 TPS2034, U15 TPS61232DRCR, U16 TPS61232DRCR, U2 TPS2034, U3 TPS2034, U4 TPS2034, U5 TPS2034, U6 TPS2034, U7 TPS2034, U8 TPS2034, U9 TPS61023DRLR

Commit message: EPS Routing
Parts:
- moved R1 82.7 mm to (129.2, 60.3)
- moved U1 80.6 mm to (133.0, 62.3), turned to -90 degrees
- moved C9 79.2 mm to (136.8, 64.3)
- moved C1 73.8 mm to (136.9, 60.3), turned to -90 degrees
- moved R3 54.8 mm to (190.0, 80.6)
- moved C10 54.8 mm to (199.4, 64.5)
- moved C12 54.8 mm to (200.4, 88.6)
- moved C2 54.8 mm to (189.8, 64.5)
- moved C4 54.8 mm to (190.8, 88.6)
- moved R2 54.8 mm to (189.8, 69.2)
- moved R4 54.8 mm to (190.8, 93.2)
- moved U2 54.8 mm to (194.6, 66.4)
- moved U4 54.8 mm to (195.6, 90.4)
- moved C11 54.8 mm to (199.7, 75.9)
- moved C3 54.8 mm to (190.0, 75.9)
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Routing:
- net PWR_LCL_1: track 0.00 -> 29.2 mm
- net ENA_LCL_1: track 0.00 -> 26.9 mm
- net Net-(U12-CE): track 0.00 -> 18.1 mm
- net Net-(U11-CE): track 0.00 -> 17.8 mm, vias 0 -> 2
- net KS_OPEN: track 0.00 -> 17.6 mm
- net Net-(U12-PSEL): track 0.00 -> 15.8 mm
- net Net-(U11-PSEL): track 0.00 -> 15.6 mm, vias 0 -> 2
- net Net-(U12-ISET2): track 0.00 -> 13.5 mm
- net Net-(U11-ISET2): track 0.00 -> 13.3 mm, vias 0 -> 2
- net Net-(D13-K): track 0.00 -> 10.7 mm, vias 0 -> 2
- net Net-(D15-K): track 0.00 -> 9.62 mm
- net Net-(D14-K): track 0.00 -> 8.98 mm, vias 0 -> 2
- net Net-(D15-A): track 0.00 -> 8.37 mm
- net Net-(D13-A): track 0.00 -> 8.35 mm
- net Net-(D16-K): track 0.00 -> 8.06 mm
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- added copper zone on B.Cu, net +BATT
- added copper zone on B.Cu, net /VIN
- added copper zone on B.Cu, net /VOUT
- added copper zone on B.Cu, net CHARGE
- added copper zone on F.Cu, net ENA_LCL_1
- added copper zone on B.Cu, net GND
- added copper zone on F.Cu, net Net-(D1-A)
- added copper zone on F.Cu, net Net-(D10-A)
- added copper zone on F.Cu, net Net-(D11-A)
- added copper zone on F.Cu, net Net-(D3-A)
- added copper zone on F.Cu, net Net-(D5-A)
- added copper zone on F.Cu, net Net-(D7-A)
- added copper zone on B.Cu, net Net-(L3-Pad2)
- added copper zone on B.Cu, net Net-(U15-EN)
- added copper zone on B.Cu, net Net-(U9-SW)
- added copper zone on F.Cu, net PWR_LCL_1
