File: LibreCube PCDU/My version/src/electrical/my_pcdu_v1.kicad_pcb (KiCad board)
At the start: 4 copper layers, 90.2 x 95.9 mm, 137 parts, among them J1 Conn_01x02, J2 Conn_01x02, J3 Conn_01x02, J4 Conn_01x02, J5 Conn_01x02, J6 Conn_01x02, J7 Conn_01x02, J8 USB_C_Receptacle_PowerOnly_6P, M1 MountingHole, M2 MountingHole, M3 MountingHole, M4 MountingHole, U1 TPS2034, U10 TPS61023DRLR, U11 BQ24032ARHLRG4, U12 BQ24032ARHLRG4, U13 TPS2034, U14 TPS2034, U15 TPS61232DRCR, U16 TPS61232DRCR, U2 TPS2034, U3 TPS2034, U4 TPS2034, U5 TPS2034, U6 TPS2034, U7 TPS2034, U8 TPS2034, U9 TPS61023DRLR

Commit message: PCDU finished
Parts:
- moved R29 171.5 mm to (107.5, 43.2), turned to 180 degrees
- moved D19 164.7 mm to (111.0, 43.2), turned to 0 degrees
- moved R5 138.8 mm to (86.6, 60.3)
- moved U5 138.0 mm to (90.3, 62.3), turned to -90 degrees
- moved C13 137.7 mm to (94.1, 64.3)
- moved J7 136.0 mm to (152.4, 42.9), turned to -90 degrees
- moved R6 133.9 mm to (97.2, 60.3)
- moved U6 132.7 mm to (100.9, 62.3), turned to -90 degrees
- moved C14 131.9 mm to (104.8, 64.3)
- moved R7 131.4 mm to (107.8, 60.3)
- moved R8 130.5 mm to (118.4, 60.3)
- moved C5 130.1 mm to (94.1, 60.3), turned to -90 degrees
- moved U7 129.5 mm to (111.6, 62.3), turned to -90 degrees
- moved C15 128.3 mm to (115.4, 64.3)
- moved U8 128.1 mm to (122.2, 62.3), turned to -90 degrees
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Connections:
- U11 pad 22: (no net) -> GND
- U11 pad 23: (no net) -> GND
- U11 pad 24: (no net) -> GND
- U11 pad 25: (no net) -> GND
- U11 pad 26: (no net) -> GND
- U11 pad 27: (no net) -> GND
- U11 pad 28: (no net) -> GND
- U11 pad 29: (no net) -> GND
- U12 pad 22: (no net) -> GND
- U12 pad 23: (no net) -> GND
- U12 pad 24: (no net) -> GND
- U12 pad 25: (no net) -> GND
- U12 pad 26: (no net) -> GND
- U12 pad 27: (no net) -> GND
- U12 pad 28: (no net) -> GND
- U12 pad 29: (no net) -> GND
Routing:
- net GND: track 0.00 -> 107.3 mm, vias 30 -> 85
- net KS_OPEN: track 17.6 -> 120.3 mm, vias 0 -> 1
- net PWR_LCL_6: track 0.00 -> 94.4 mm
- net CHARGE: track 0.00 -> 94.0 mm, vias 0 -> 24
- net PWR_LCL_5: track 0.00 -> 80.8 mm
- net ENA_LCL_5: track 0.00 -> 58.0 mm
- net ENA_LCL_6: track 0.00 -> 50.0 mm
- net +BATT: track 0.00 -> 44.5 mm, vias 0 -> 12
- net PWR_LCL_7: track 0.00 -> 43.6 mm
- net ENA_LCL_7: track 0.00 -> 41.2 mm
- net PWR_LCL_8: track 0.00 -> 37.2 mm
- net ENA_LCL_8: track 0.00 -> 33.7 mm
- net PWR_LCL_4: track 0.00 -> 23.9 mm
- net PWR_LCL_2: track 0.00 -> 20.8 mm
- net ENA_LCL_2: track 0.00 -> 17.8 mm
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- added copper zone on F.Cu, net +5V
- added copper zone on F.Cu, net +BATT
- added copper zone on F.Cu, net CHARGE
- added copper zone on F.Cu, net ENA_LCL_2
- added copper zone on F.Cu, net ENA_LCL_3
- added copper zone on F.Cu, net ENA_LCL_4
- added copper zone on F.Cu, net ENA_LCL_5
- added copper zone on F.Cu, net ENA_LCL_6
- added copper zone on F.Cu, net ENA_LCL_7
- added copper zone on F.Cu, net ENA_LCL_8
- added copper zone on F.Cu, net GND
- added copper zone on In1.Cu, net GND
- added copper zone on In2.Cu, net GND
- added copper zone on B.Cu, net Net-(L4-Pad2)
- added copper zone on F.Cu, net PWR_LCL_2
- added copper zone on F.Cu, net PWR_LCL_3
- added copper zone on F.Cu, net PWR_LCL_4
- added copper zone on F.Cu, net PWR_LCL_5
- added copper zone on F.Cu, net PWR_LCL_6
- added copper zone on F.Cu, net PWR_LCL_7
- added copper zone on F.Cu, net PWR_LCL_8
Other:
- rule pad_to_mask_clearance: 0 -> 0.038

Commit message: PCDU Complete
Routing:
- net CHARGE: track 94.0 -> 94.9 mm
- net GND: vias 85 -> 305
Other:
- board text added: "{ "ViaStitching": "0.2", "stitch_zone_0": { "HSpacing": "2.5", "VSpacing": "2.5", "HOffset": "0", "VOffset": "0", "Clearance": "0", "Randomize": false } }"
- board text added: "{ "ViaStitching": "0.2", "stitch_zone_0": { "HSpacing": "2.5", "VSpacing": "2.5", "HOffset": "0", "VOffset": "0", "Clearance": "0.2", "Randomize": false } }"
- board text added: "{ "ViaStitching": "0.2", "stitch_zone_0": { "HSpacing": "2.5", "VSpacing": "2.5", "HOffset": "1.25", "VOffset": "1.25", "Clearance": "0", "Randomize": false } }"
- board text added: "{ "ViaStitching": "0.2", "stitch_zone_0": { "HSpacing": "2.54", "VSpacing": "2.54", "HOffset": "0", "VOffset": "0", "Clearance": "0.2", "Randomize": false } }"
- board text added: "{ "ViaStitching": "0.2", "stitch_zone_0": { "HSpacing": "2.54", "VSpacing": "2.54", "HOffset": "1.27", "VOffset": "1.27", "Clearance": "0.2", "Randomize": false } }"
